File: BatteryBusDetection.kicad_sch (KiCad schematic)
At the start: 12 parts, among them U1 S-8209AAA-T8T1U, U2 S-8209AAA-T8T1U

Commit message: First pass at new schematics and board
Parts:
- C1, C2, C3, C4: footprint (none) -> Capacitor_SMD:C_0603_1608Metric
- R1, R2, R4, R5, R6, R7: footprint (none) -> Resistor_SMD:R_0603_1608Metric
- U1, U2: footprint TSSOP8-E-PKG_FT008-A-P-SD-1.2_ABL -> Battery-Board:TSSOP8-E-PKG_FT008-A-P-SD-1.2_ABL
Connections:
- net CHARGE_ENABLE renamed CHARGE_EN
- net DISCHARGE_ENABLE renamed DISCHARGE_EN
Changed lines of the file:
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@@
 		)
 	)
-	(hierarchical_label "CHARGE_ENABLE"
+	(hierarchical_label "CHARGE_EN"
 		(shape output)
 		(at 237.49 81.28 0)
@@
 		)
 	)
-	(hierarchical_label "DISCHARGE_ENABLE"
+	(hierarchical_label "DISCHARGE_EN"
 		(shape output)
 		(at 237.49 83.82 0)
@@
 			)
 		)
-		(property "Footprint" ""
+		(property "Footprint" "Resistor_SMD:R_0603_1608Metric"
 			(at 161.29 102.87 0)
 			(effects
@@
 			)
 		)
-		(property "Footprint" ""
+		(property "Footprint" "Resistor_SMD:R_0603_1608Metric"
 			(at 102.87 105.41 0)
 			(effects
@@
 			)
 		)
-		(property "Footprint" ""
+		(property "Footprint" "Capacitor_SMD:C_0603_1608Metric"
 			(at 102.87 124.46 0)
 			(effects
@@
 			)
 		)
-		(property "Footprint" ""
+		(property "Footprint" "Resistor_SMD:R_0603_1608Metric"
 			(at 92.71 124.46 0)
 			(effects
@@
 			)
 		)
-		(property "Footprint" "TSSOP8-E-PKG_FT008-A-P-SD-1.2_ABL"
+		(property "Footprint" "Battery-Board:TSSOP8-E-PKG_FT008-A-P-SD-1.2_ABL"
 			(at 116.84 111.76 0)
 			(effects
@@
 			)
 		)
-		(property "Footprint" ""
+		(property "Footprint" "Capacitor_SMD:C_0603_1608Metric"
 			(at 182.88 91.44 0)
 			(effects
@@
 			)
 		)
-		(property "Footprint" ""
+		(property "Footprint" "Resistor_SMD:R_0603_1608Metric"
 			(at 171.45 69.85 0)
 			(effects
@@
 			)
 		)
-		(property "Footprint" ""
+		(property "Footprint" "Capacitor_SMD:C_0603_1608Metric"
 			(at 171.45 91.44 0)
 			(effects
@@
 			)
 		)
-		(property "Footprint" ""
+		(property "Footprint" "Capacitor_SMD:C_0603_1608Metric"
 			(at 114.3 124.46 0)
 			(effects
@@
 			)
 		)
-		(property "Footprint" ""
+		(property "Footprint" "Resistor_SMD:R_0603_1608Metric"
 			(at 167.64 111.76 0)
 			(effects
@@
 			)
 		)
-		(property "Footprint" "TSSOP8-E-PKG_FT008-A-P-SD-1.2_ABL"
+		(property "Footprint" "Battery-Board:TSSOP8-E-PKG_FT008-A-P-SD-1.2_ABL"
 			(at 185.42 78.74 0)
 			(effects
@@
 			)
 		)
-		(property "Footprint" ""
+		(property "Footprint" "Resistor_SMD:R_0603_1608Metric"
 			(at 83.82 124.46 0)
 			(effects
