File: BatteryBusDetection.kicad_sch (KiCad schematic)
At the start: 12 parts, among them U1 S-8209AAA-T8T1U, U2 S-8209AAA-T8T1U

Commit message: making a few changes
Other:
- title: Argus Batteryboard -> Batteryboard
Changed lines of the file:
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@@
 	(paper "USLetter")
 	(title_block
-		(title "Argus Batteryboard")
-		(date "2026-04-14")
-		(rev "v3.2")
+		(title "Batteryboard")
+		(date "2026-08-21")
+		(rev "v4.0")
 		(company "Carnegie Mellon University")
-		(comment 1 "M. Holliday")
-		(comment 2 "N. Khera")
-		(comment 3 "V. Rajesh")
+		(comment 1 "N. Khera")
+		(comment 2 "V. Rajesh")
+		(comment 3 "S. Farhan")
 	)
 	(rectangle

Commit message: routing
Parts:
- renumbered C3 to C1, C4 to C2, C1 to C3, C2 to C4, R6 to R1, R4 to R2, R5 to R3, R3 to R4, R1 to R5, R2 to R6, U2 to U1, U1 to U2
Changed lines of the file:
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@@
 		(in_pos_files yes)
 		(dnp no)
-		(property "Reference" "R4"
+		(property "Reference" "R2"
 			(at 143.51 91.694 0)
 			(show_name no)
@@
 			(project "Avionics-BatteryBoard"
 				(path "/b6fd875d-6e05-4440-9a05-0f0aa046a0ef/7ba9fa06-6a7f-47d4-99e7-e1daf0ec12b6"
-					(reference "R4")
+					(reference "R2")
 					(unit 1)
 				)
@@
 		(in_pos_files yes)
 		(dnp no)
-		(property "Reference" "R3"
+		(property "Reference" "R4"
 			(at 87.63 105.664 0)
 			(show_name no)
@@
 			(project "Avionics-BatteryBoard"
 				(path "/b6fd875d-6e05-4440-9a05-0f0aa046a0ef/7ba9fa06-6a7f-47d4-99e7-e1daf0ec12b6"
-					(reference "R3")
+					(reference "R4")
 					(unit 1)
 				)
@@
 		(in_pos_files yes)
 		(dnp no)
-		(property "Reference" "C1"
+		(property "Reference" "C3"
 			(at 88.392 124.714 0)
 			(show_name no)
@@
 			(project "Avionics-BatteryBoard"
 				(path "/b6fd875d-6e05-4440-9a05-0f0aa046a0ef/7ba9fa06-6a7f-47d4-99e7-e1daf0ec12b6"
-					(reference "C1")
+					(reference "C3")
 					(unit 1)
 				)
@@
 		(in_pos_files yes)
 		(dnp no)
-		(property "Reference" "R2"
+		(property "Reference" "R6"
 			(at 81.28 124.714 0)
 			(show_name no)
@@
 			(project "Avionics-BatteryBoard"
 				(path "/b6fd875d-6e05-4440-9a05-0f0aa046a0ef/7ba9fa06-6a7f-47d4-99e7-e1daf0ec12b6"
-					(reference "R2")
+					(reference "R6")
 					(unit 1)
 				)
@@
 		(in_pos_files yes)
 		(dnp no)
-		(property "Reference" "U1"
+		(property "Reference" "U2"
 			(at 119.38 104.394 0)
 			(show_name no)
@@
 			(project "Avionics-BatteryBoard"
 				(path "/b6fd875d-6e05-4440-9a05-0f0aa046a0ef/7ba9fa06-6a7f-47d4-99e7-e1daf0ec12b6"
-					(reference "U1")
+					(reference "U2")
 					(unit 1)
 				)
@@
 		(in_pos_files yes)
 		(dnp no)
-		(property "Reference" "C4"
+		(property "Reference" "C2"
 			(at 167.132 91.694 0)
 			(show_name no)
@@
 			(project "Avionics-BatteryBoard"
 				(path "/b6fd875d-6e05-4440-9a05-0f0aa046a0ef/7ba9fa06-6a7f-47d4-99e7-e1daf0ec12b6"
-					(reference "C4")
+					(reference "C2")
 					(unit 1)
 				)
@@
 		(in_pos_files yes)
 		(dnp no)
-		(property "Reference" "R6"
+		(property "Reference" "R1"
 			(at 156.21 70.104 0)
 			(show_name no)
@@
 			(project "Avionics-BatteryBoard"
 				(path "/b6fd875d-6e05-4440-9a05-0f0aa046a0ef/7ba9fa06-6a7f-47d4-99e7-e1daf0ec12b6"
-					(reference "R6")
+					(reference "R1")
 					(unit 1)
 				)
@@
 		(in_pos_files yes)
 		(dnp no)
-		(property "Reference" "C3"
+		(property "Reference" "C1"
 			(at 156.972 91.694 0)
 			(show_name no)
@@
 			(project "Avionics-BatteryBoard"
 				(path "/b6fd875d-6e05-4440-9a05-0f0aa046a0ef/7ba9fa06-6a7f-47d4-99e7-e1daf0ec12b6"
-					(reference "C3")
+					(reference "C1")
 					(unit 1)
 				)
@@
 		(in_pos_files yes)
 		(dnp no)
-		(property "Reference" "C2"
+		(property "Reference" "C4"
 			(at 98.552 124.714 0)
 			(show_name no)
@@
 			(project "Avionics-BatteryBoard"
 				(path "/b6fd875d-6e05-4440-9a05-0f0aa046a0ef/7ba9fa06-6a7f-47d4-99e7-e1daf0ec12b6"
-					(reference "C2")
+					(reference "C4")
 					(unit 1)
 				)
@@
 		(in_pos_files yes)
 		(dnp no)
-		(property "Reference" "R5"
+		(property "Reference" "R3"
 			(at 149.86 91.694 0)
 			(show_name no)
@@
 			(project "Avionics-BatteryBoard"
 				(path "/b6fd875d-6e05-4440-9a05-0f0aa046a0ef/7ba9fa06-6a7f-47d4-99e7-e1daf0ec12b6"
-					(reference "R5")
+					(reference "R3")
 					(unit 1)
 				)
@@
 		(in_pos_files yes)
 		(dnp no)
-		(property "Reference" "U2"
+		(property "Reference" "U1"
 			(at 187.96 71.374 0)
 			(show_name no)
@@
 			(project "Avionics-BatteryBoard"
 				(path "/b6fd875d-6e05-4440-9a05-0f0aa046a0ef/7ba9fa06-6a7f-47d4-99e7-e1daf0ec12b6"
-					(reference "U2")
+					(reference "U1")
 					(unit 1)
 				)
@@
 		(in_pos_files yes)
 		(dnp no)
-		(property "Reference" "R1"
+		(property "Reference" "R5"
 			(at 74.93 124.714 0)
 			(show_name no)
@@
 			(project "Avionics-BatteryBoard"
 				(path "/b6fd875d-6e05-4440-9a05-0f0aa046a0ef/7ba9fa06-6a7f-47d4-99e7-e1daf0ec12b6"
-					(reference "R1")
-					(unit 1)
-				)
+					(reference "R5")
+					(unit 1)
+				)
