File: IOExpander.kicad_sch (KiCad schematic)
At the start: 2 parts, among them U12 PCA9536D

Commit message: First pass at new schematics and board
Parts:
- added R46, R48: 100k, Resistor_SMD:R_0603_1608Metric, symbol Device:R_Small
- added R47, R49: 100k, Capacitor_SMD:C_0603_1608Metric, symbol Device:R_Small
- C16: footprint (none) -> Capacitor_SMD:C_0603_1608Metric
Connections:
- net GND: now also R46.1, R47.1, R48.1, R49.1
- net IO0: now also R46.2
- net IO1: now also R48.2
- net IO2: now also R47.2
- net IO3: now also R49.2
