File: BatteryBoard.kicad_pcb (KiCad board)
At the start: 4 copper layers, 90.2 x 95.9 mm, 133 parts, among them J1 Keystone-1048, J10 200528-0100, J5 Keystone-1042, J6 Keystone-1042, J7 1824543, J8 Conn_01x06, J9 Keystone-1048, Q1 NX3008NBKS, Q2 MBT2222ADW1T1, Q3 NX3008NBKS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

Commit message: Changes for lib refactor
Parts:
- J1, J9: footprint Battery-Board:BAT_1048 -> Argus-Misc:BAT_1048
- J5, J6: footprint Battery-Board:Keystone_1042 -> Argus-Misc:Keystone_1042
- J7: footprint Battery-Board:1824543 -> Argus-Connectors:1824543
- U1, U2: footprint Battery-Board:TSSOP8-E-PKG_FT008-A-P-SD-1.2_ABL -> Argus-IC:TSSOP8-E-PKG_FT008-A-P-SD-1.2_ABL
- U3: footprint Battery-Board:21-0137_T1433&plus_2C_MXM -> Argus-IC:21-0137_T1433&plus_2C_MXM
- U4, U5, U6, U7: footprint Battery-Board:MOSFET_7DP-T1-GE3_VIS -> Argus-Misc:MOSFET_7DP-T1-GE3_VIS

Commit message: Fixes from feedback
Connections:
- C10 pad 1: Net-(U8-VIN) -> SYSTEM_VDD
- U4 pad 5: Net-(U4-D-Pad5) -> Net-(U9-VIN)
- U4 pad 6: Net-(U4-D-Pad5) -> Net-(U9-VIN)
- U4 pad 7: Net-(U4-D-Pad5) -> Net-(U9-VIN)
- U4 pad 8: Net-(U4-D-Pad5) -> Net-(U9-VIN)
- U5 pad 5: Net-(U4-D-Pad5) -> Net-(U9-VIN)
- U5 pad 6: Net-(U4-D-Pad5) -> Net-(U9-VIN)
- U5 pad 7: Net-(U4-D-Pad5) -> Net-(U9-VIN)
- U5 pad 8: Net-(U4-D-Pad5) -> Net-(U9-VIN)
- U8 pad 1: Net-(U8-VIN) -> SYSTEM_VDD
Routing:
- net Net-(U9-VIN): track 2.93 -> 7.88 mm
- net SYSTEM_VDD: track 40.2 -> 45.2 mm
- net Net-(U8-VIN): track 2.93 -> 0.00 mm
- net GND: vias 27 -> 32
- added copper zone on B.Cu, net Net-(U9-VIN)
- removed copper zone on B.Cu, net Net-(U4-D-Pad5)
Other:
- board text added: "ARGUS-2 CMU Cubesat BatteryBoard v1"

Commit message: Added more silkscreen for mainboard connector
Other:
- board text added: "3.3V"
- board text added: "ALRT"
- board text added: "GND"
- board text added: "MAINBOARD"
- board text added: "SCL"
- board text added: "SDA"
Changed lines of the file:
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@@
 		(tags "connector Molex  top entry")
 		(property "Reference" "J10"
-			(at 0 2.61 90)
+			(at 0 -1.39 90)
 			(layer "B.SilkS")
 			(effects
@@
 		)
 	)
+	(gr_line
+		(start 106.6176 94.2304)
+		(end 106.6176 105)
+		(stroke
+			(width 0.127)
+			(type default)
+		)
+		(layer "B.SilkS")
+	)
 	(gr_rect
 		(start 96.5 111)
@@
 		(layer "B.SilkS")
 	)
+	(gr_line
+		(start 106.6176 105)
+		(end 105.5 105)
+		(stroke
+			(width 0.127)
+			(type default)
+		)
+		(layer "B.SilkS")
+	)
+	(gr_line
+		(start 106.6176 94.2304)
+		(end 105.5 94.2304)
+		(stroke
+			(width 0.127)
+			(type default)
+		)
+		(layer "B.SilkS")
+	)
 	(gr_arc
 		(start 95.3165 53.5)
@@
 		(layer "Edge.Cuts")
 	)
+	(gr_text "3.3V"
+		(at 104.1665 95.1194 0)
+		(layer "B.SilkS")
+		(effects
+			(font
+				(size 0.508 0.508)
+				(thickness 0.1016)
+				(bold yes)
+			)
+			(justify right mirror)
+		)
+	)
+	(gr_text "GND"
+		(at 104.1665 97.126 0)
+		(layer "B.SilkS")
+		(effects
+			(font
+				(size 0.508 0.508)
+				(thickness 0.1016)
+				(bold yes)
+			)
+			(justify right mirror)
+		)
+	)
+	(gr_text "GND"
+		(at 104.1665 98.1166 0)
+		(layer "B.SilkS")
+		(effects
+			(font
+				(size 0.508 0.508)
+				(thickness 0.1016)
+				(bold yes)
+			)
+			(justify right mirror)
+		)
+	)
+	(gr_text "SCL"
+		(at 104.1665 99.1326 0)
+		(layer "B.SilkS")
+		(effects
+			(font
+				(size 0.508 0.508)
+				(thickness 0.1016)
+				(bold yes)
+			)
+			(justify right mirror)
+		)
+	)
+	(gr_text "MAINBOARD"
+		(at 97 99.5 90)
+		(layer "B.SilkS")
+		(effects
+			(font
+				(size 0.635 0.635)
+				(thickness 0.1016)
+			)
+			(justify mirror)
+		)
+	)
 	(gr_text "ARGUS-2\nCMU Cubesat\nBatteryBoard v1"
 		(at 109 88.5 0)
@@
 		)
 	)
+	(gr_text "3.3V"
+		(at 104.1665 96.11 0)
+		(layer "B.SilkS")
+		(effects
+			(font
+				(size 0.508 0.508)
+				(thickness 0.1016)
+				(bold yes)
+			)
+			(justify right mirror)
+		)
+	)
+	(gr_text "GND"
+		(at 104.1665 102.1298 0)
+		(layer "B.SilkS")
+		(effects
+			(font
+				(size 0.508 0.508)
+				(thickness 0.1016)
+				(bold yes)
+			)
+			(justify right mirror)
+		)
+	)
+	(gr_text "GND"
+		(at 104.1665 104.111 0)
+		(layer "B.SilkS")
+		(effects
+			(font
+				(size 0.508 0.508)
+				(thickness 0.1016)
+				(bold yes)
+			)
+			(justify right mirror)
+		)
+	)
+	(gr_text "SDA"
+		(at 104.1665 100.1232 0)
+		(layer "B.SilkS")
+		(effects
+			(font
+				(size 0.508 0.508)
+				(thickness 0.1016)
+				(bold yes)
+			)
+			(justify right mirror)
+		)
+	)
+	(gr_text "GND"
+		(at 104.1665 103.1204 0)
+		(layer "B.SilkS")
+		(effects
+			(font
+				(size 0.508 0.508)
+				(thickness 0.1016)
+				(bold yes)
+			)
+			(justify right mirror)
+		)
+	)
+	(gr_text "ALRT"
+		(at 104.1665 101.1392 0)
+		(layer "B.SilkS")
+		(effects
+			(font
+				(size 0.508 0.508)
+				(thickness 0.1016)
+				(bold yes)
+			)
+			(justify right mirror)
+		)
+	)

Commit message: Updated silkscreen
Parts:
- added REF**: Val**, mainboard:XYZ_cubesat-bot, F.Cu at (178.0, 113.0)
