File: BatteryBoard.kicad_sch (KiCad schematic)
At the start: 8 parts, among them J1 Keystone-1042, J2 Keystone-1042, J3 Keystone-1042, J4 Keystone-1042, J5 Keystone-1042, J6 Keystone-1042, J7 1824543, J8 Conn_01x06

Commit message: First pass at new schematics and board
Parts:
- removed J1, J2, J3, J4, J5, J6: Keystone-1042, symbol Battery-Board:Keystone-1042
- removed J7: 1824543, 1824543, symbol Battery-Board:1824543
- removed J8: Conn_01x06, Connector_PinHeader_2.54mm:PinHeader_1x06_P2.54mm_Vertical, symbol Connector_Generic:Conn_01x06
- added H1, H2, H3, H4: MountingHole_Pad, MountingHole:MountingHole_3.2mm_M3_Pad_TopBottom, symbol Mechanical:MountingHole_Pad
Connections:
- net GND: now also H1.1, H2.1, H3.1, H4.1
Other:
- added sheet Battery (Battery.kicad_sch)
- added sheet Interfaces (Interfaces.kicad_sch)

Commit message: Updated version to v2.1
Other:
- company: (none) -> Carnegie Mellon University
- title: (none) -> Argus Batteryboard
Changed lines of the file:
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@@
 	(generator_version "8.0")
 	(paper "A4")
+	(title_block
+		(title "Argus Batteryboard")
+		(date "2024-11-19")
+		(rev "v2.1")
+		(company "Carnegie Mellon University")
+		(comment 1 "M. Holliday")
+		(comment 2 "N. Khera")
+		(comment 3 "V. Rajesh")
+	)
 	(junction
 		(at 200.66 121.92)

Commit message: v2.1 (v3?) Partial Updates
Connections:
- no-connect marks 0 -> 1
Other:
- removed sheet Battery Temperature Protection1
- removed sheet I2C Protection
- removed sheet I2C Protection1
- sheet Battery ports: added BATT_M, BATT_N, BATT_P; removed BATT0, BATT1, BATT2
- sheet Battery Bus Detection ports: added BATT_M, BATT_N, BATT_P; removed BATT0, BATT1, BATT2
- sheet Battery Bus Protection ports: added BATT_P; removed BATT2
- sheet Battery Monitor ports: added BATT_M, BATT_N, BATT_P; removed BATT0, BATT1, BATT2
- sheet Battery Temperature Protection ports: added CB-RESET, HEATER_ENABLE0, HEATER_ENABLE1, ON/~{OFF}, ~{FAULT}; removed HEATER_ENABLE
- sheet IO Expander ports: added IO4, IO5, IO6, IO7; removed none
- note added: "Could put ALERT ON IO5"
- note added: "Could put all GPIO ON FPC"
- moved on the sheet: H1, H2, H3, H4
