File: I2CProtection.kicad_sch (KiCad schematic)
At the start: 18 parts, among them Q1 NX3008NBKS, Q2 MBT2222ADW1T1, Q3 NX3008NBKS, Q4 MBT2222ADW1T1

Commit message: First pass at new schematics and board
Parts:
- renumbered C12 to C14, C13 to C15, Q1 to Q5, Q2 to Q6, Q3 to Q7, Q4 to Q8, R14 to R28, R15 to R29, R16 to R30, R17 to R31, R18 to R32, R19 to R33, R20 to R34, R21 to R35, R22 to R36, R23 to R37, R24 to R38, R25 to R39
Changed lines of the file:
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@@
 		(on_board yes)
 		(dnp no)
-		(property "Reference" "Q3"
+		(property "Reference" "Q7"
 			(at 167.767 99.06 0)
 			(effects
@@
 		(on_board yes)
 		(dnp no)
-		(property "Reference" "Q4"
+		(property "Reference" "Q8"
 			(at 172.72 72.009 90)
 			(effects
@@
 		(on_board yes)
 		(dnp no)
-		(property "Reference" "#PWR011"
+		(property "Reference" "#PWR020"
 			(at 177.8 115.57 0)
 			(effects
@@
 		(on_board yes)
 		(dnp no)
-		(property "Reference" "#PWR09"
+		(property "Reference" "#PWR018"
 			(at 162.56 90.17 0)
 			(effects
@@
 		(on_board yes)
 		(dnp no)
-		(property "Reference" "R20"
+		(property "Reference" "R34"
 			(at 144.78 142.621 90)
 			(effects
@@
 		(on_board yes)
 		(dnp no)
-		(property "Reference" "#PWR06"
+		(property "Reference" "#PWR015"
 			(at 120.65 90.17 0)
 			(effects
@@
 		(on_board yes)
 		(dnp no)
-		(property "Reference" "Q2"
+		(property "Reference" "Q6"
 			(at 130.81 72.009 90)
 			(effects
@@
 		(on_board yes)
 		(dnp no)
-		(property "Reference" "R25"
+		(property "Reference" "R39"
 			(at 178.816 91.694 0)
 			(effects
@@
 		(on_board yes)
 		(dnp no)
-		(property "Reference" "R23"
+		(property "Reference" "R37"
 			(at 171.704 56.134 0)
 			(effects
@@
 		(on_board yes)
 		(dnp no)
-		(property "Reference" "R16"
+		(property "Reference" "R30"
 			(at 129.667 56.134 0)
 			(effects
@@
 		(on_board yes)
 		(dnp no)
-		(property "Reference" "R21"
+		(property "Reference" "R35"
 			(at 161.29 74.676 90)
 			(effects
@@
 		(on_board yes)
 		(dnp no)
-		(property "Reference" "#PWR010"
+		(property "Reference" "#PWR019"
 			(at 172.72 57.15 0)
 			(effects
@@
 		(on_board yes)
 		(dnp no)
-		(property "Reference" "#PWR08"
+		(property "Reference" "#PWR017"
 			(at 135.89 115.57 0)
 			(effects
@@
 		(on_board yes)
 		(dnp no)
-		(property "Reference" "C13"
+		(property "Reference" "C15"
 			(at 180.594 101.854 0)
 			(effects
@@
 		(on_board yes)
 		(dnp no)
-		(property "Reference" "Q1"
+		(property "Reference" "Q5"
 			(at 125.476 99.06 0)
 			(effects
@@
 		(on_board yes)
 		(dnp no)
-		(property "Reference" "R22"
+		(property "Reference" "R36"
 			(at 163.576 89.154 0)
 			(effects
@@
 		(on_board yes)
 		(dnp no)
-		(property "Reference" "R24"
+		(property "Reference" "R38"
 			(at 178.816 62.484 0)
 			(effects
@@
 		(on_board yes)
 		(dnp no)
-		(property "Reference" "C12"
+		(property "Reference" "C14"
 			(at 138.684 101.854 0)
 			(effects
@@
 		(on_board yes)
 		(dnp no)
-		(property "Reference" "Q1"
+		(property "Reference" "Q5"
 			(at 110.236 93.98 0)
 			(effects
@@
 		(on_board yes)
 		(dnp no)
-		(property "Reference" "#PWR07"
+		(property "Reference" "#PWR016"
 			(at 130.81 55.88 0)
 			(effects
@@
 		(on_board yes)
 		(dnp no)
-		(property "Reference" "Q2"
+		(property "Reference" "Q6"
 			(at 130.81 89.408 90)
 			(effects
@@
 		(on_board yes)
 		(dnp no)
-		(property "Reference" "R18"
+		(property "Reference" "R32"
 			(at 137.033 91.694 0)
 			(effects
@@
 		(on_board yes)
 		(dnp no)
-		(property "Reference" "Q4"
+		(property "Reference" "Q8"
 			(at 172.72 89.408 90)
 			(effects
@@
 		(on_board yes)
 		(dnp no)
-		(property "Reference" "R14"
+		(property "Reference" "R28"
 			(at 119.38 74.676 90)
 			(effects
@@
 		(on_board yes)
 		(dnp no)
-		(property "Reference" "Q3"
+		(property "Reference" "Q7"
 			(at 152.146 93.98 0)
 			(effects
@@
 		(on_board yes)
 		(dnp no)
-		(property "Reference" "R17"
+		(property "Reference" "R31"
 			(at 137.033 62.484 0)
 			(effects
@@
 		(on_board yes)
 		(dnp no)
-		(property "Reference" "R19"
+		(property "Reference" "R33"
 			(at 144.78 134.874 90)
 			(effects
@@
 		(on_board yes)
 		(dnp no)
-		(property "Reference" "R15"
+		(property "Reference" "R29"
 			(at 121.793 89.154 0)
 			(effects

Commit message: Fixes from feedback
Parts:
- Q5, Q7: symbol BatteryBoard:NX3008NBKS -> Device:Q_Dual_NMOS_S1G1D2S2G2D1

Commit message: v2.1 (v3?) Partial Updates
Parts:
- R61: renamed from R30; value 10K -> 10k
- R62: renamed from R31; value 10K -> 10k
- R64: renamed from R29; value 100K -> 100k
- R65: renamed from R32; value 200K -> 200k
- R66: renamed from R37; value 10K -> 10k
- R67: renamed from R38; value 10K -> 10k
- R69: renamed from R36; value 100K -> 100k
- R70: renamed from R39; value 200K -> 200k
- R71: renamed from R33; now not fitted
- R72: renamed from R34; now not fitted
- renumbered Q5 to Q15, Q6 to Q16, Q7 to Q17, Q8 to Q18, R28 to R63, R35 to R68
Other:
- company: (none) -> Carnegie Mellon University
- title: (none) -> Argus Batteryboard

Commit message: More updates
Parts:
- R71, R72: value DNI (0R) -> 0R
Changed lines of the file:
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@@
 	(title_block
 		(title "Argus Batteryboard")
-		(date "2024-12-06")
-		(rev "v2.1")
+		(date "2025-01-08")
+		(rev "v3.0")
 		(company "Carnegie Mellon University")
 		(comment 1 "M. Holliday")
@@
 					(unit 2)
 				)
-				(path "/b6fd875d-6e05-4440-9a05-0f0aa046a0ef/e121e58f-b773-45d1-af83-1cd1570c2804/b948d429-f108-462e-8f18-75ba0a87c593"
-					(reference "Q21")
-					(unit 2)
-				)
 			)
 		)
@@
 					(unit 2)
 				)
-				(path "/b6fd875d-6e05-4440-9a05-0f0aa046a0ef/e121e58f-b773-45d1-af83-1cd1570c2804/b948d429-f108-462e-8f18-75ba0a87c593"
-					(reference "Q22")
-					(unit 2)
-				)
 			)
 		)
@@
 					(unit 1)
 				)
-				(path "/b6fd875d-6e05-4440-9a05-0f0aa046a0ef/e121e58f-b773-45d1-af83-1cd1570c2804/b948d429-f108-462e-8f18-75ba0a87c593"
-					(reference "#PWR018")
-					(unit 1)
-				)
 			)
 		)
@@
 					(unit 1)
 				)
-				(path "/b6fd875d-6e05-4440-9a05-0f0aa046a0ef/e121e58f-b773-45d1-af83-1cd1570c2804/b948d429-f108-462e-8f18-75ba0a87c593"
-					(reference "#PWR016")
-					(unit 1)
-				)
 			)
 		)
@@
 			)
 		)
-		(property "Value" "DNI (0R)"
+		(property "Value" "0R"
 			(at 144.78 147.193 90)
 			(effects
@@
 				(path "/b6fd875d-6e05-4440-9a05-0f0aa046a0ef/ad142cc2-d77f-4a6c-99c2-d9e17f4c27ae/8631bf3a-5019-45d5-a8fe-6e53ccedb3c2"
 					(reference "R72")
-					(unit 1)
-				)
-				(path "/b6fd875d-6e05-4440-9a05-0f0aa046a0ef/e121e58f-b773-45d1-af83-1cd1570c2804/b948d429-f108-462e-8f18-75ba0a87c593"
-					(reference "R91")
 					(unit 1)
 				)
@@
 				(path "/b6fd875d-6e05-4440-9a05-0f0aa046a0ef/ad142cc2-d77f-4a6c-99c2-d9e17f4c27ae/8631bf3a-5019-45d5-a8fe-6e53ccedb3c2"
 					(reference "#PWR02")
-					(unit 1)
-				)
-				(path "/b6fd875d-6e05-4440-9a05-0f0aa046a0ef/e121e58f-b773-45d1-af83-1cd1570c2804/b948d429-f108-462e-8f18-75ba0a87c593"
-					(reference "#PWR09")
 					(unit 1)
 				)
@@
 					(unit 2)
 				)
-				(path "/b6fd875d-6e05-4440-9a05-0f0aa046a0ef/e121e58f-b773-45d1-af83-1cd1570c2804/b948d429-f108-462e-8f18-75ba0a87c593"
-					(reference "Q20")
-					(unit 2)
-				)
 			)
 		)
@@
 					(unit 1)
 				)
-				(path "/b6fd875d-6e05-4440-9a05-0f0aa046a0ef/e121e58f-b773-45d1-af83-1cd1570c2804/b948d429-f108-462e-8f18-75ba0a87c593"
-					(reference "R89")
-					(unit 1)
-				)
 			)
 		)
@@
 					(unit 1)
 				)
-				(path "/b6fd875d-6e05-4440-9a05-0f0aa046a0ef/e121e58f-b773-45d1-af83-1cd1570c2804/b948d429-f108-462e-8f18-75ba0a87c593"
-					(reference "R85")
-					(unit 1)
-				)
 			)
 		)
@@
 					(unit 1)
 				)
-				(path "/b6fd875d-6e05-4440-9a05-0f0aa046a0ef/e121e58f-b773-45d1-af83-1cd1570c2804/b948d429-f108-462e-8f18-75ba0a87c593"
-					(reference "R80")
-					(unit 1)
-				)
 			)
 		)
@@
 					(unit 1)
 				)
-				(path "/b6fd875d-6e05-4440-9a05-0f0aa046a0ef/e121e58f-b773-45d1-af83-1cd1570c2804/b948d429-f108-462e-8f18-75ba0a87c593"
-					(reference "R87")
-					(unit 1)
-				)
 			)
 		)
@@
 					(unit 1)
 				)
-				(path "/b6fd875d-6e05-4440-9a05-0f0aa046a0ef/e121e58f-b773-45d1-af83-1cd1570c2804/b948d429-f108-462e-8f18-75ba0a87c593"
-					(reference "#PWR017")
-					(unit 1)
-				)
 			)
 		)
@@
 					(unit 1)
 				)
-				(path "/b6fd875d-6e05-4440-9a05-0f0aa046a0ef/e121e58f-b773-45d1-af83-1cd1570c2804/b948d429-f108-462e-8f18-75ba0a87c593"
-					(reference "#PWR015")
-					(unit 1)
-				)
 			)
 		)
@@
 				(path "/b6fd875d-6e05-4440-9a05-0f0aa046a0ef/ad142cc2-d77f-4a6c-99c2-d9e17f4c27ae/8631bf3a-5019-45d5-a8fe-6e53ccedb3c2"
 					(reference "C15")
-					(unit 1)
-				)
-				(path "/b6fd875d-6e05-4440-9a05-0f0aa046a0ef/e121e58f-b773-45d1-af83-1cd1570c2804/b948d429-f108-462e-8f18-75ba0a87c593"
-					(reference "C18")
 					(unit 1)
 				)
@@
 					(unit 2)
 				)
-				(path "/b6fd875d-6e05-4440-9a05-0f0aa046a0ef/e121e58f-b773-45d1-af83-1cd1570c2804/b948d429-f108-462e-8f18-75ba0a87c593"
-					(reference "Q19")
-					(unit 2)
-				)
 			)
 		)
@@
 					(unit 1)
 				)
-				(path "/b6fd875d-6e05-4440-9a05-0f0aa046a0ef/e121e58f-b773-45d1-af83-1cd1570c2804/b948d429-f108-462e-8f18-75ba0a87c593"
-					(reference "R88")
-					(unit 1)
-				)
 			)
 		)
@@
 					(unit 1)
 				)
-				(path "/b6fd875d-6e05-4440-9a05-0f0aa046a0ef/e121e58f-b773-45d1-af83-1cd1570c2804/b948d429-f108-462e-8f18-75ba0a87c593"
-					(reference "R86")
-					(unit 1)
-				)
 			)
 		)
@@
 				(path "/b6fd875d-6e05-4440-9a05-0f0aa046a0ef/ad142cc2-d77f-4a6c-99c2-d9e17f4c27ae/8631bf3a-5019-45d5-a8fe-6e53ccedb3c2"
 					(reference "C14")
-					(unit 1)
-				)
-				(path "/b6fd875d-6e05-4440-9a05-0f0aa046a0ef/e121e58f-b773-45d1-af83-1cd1570c2804/b948d429-f108-462e-8f18-75ba0a87c593"
-					(reference "C17")
 					(unit 1)
 				)
@@
 					(unit 1)
 				)
-				(path "/b6fd875d-6e05-4440-9a05-0f0aa046a0ef/e121e58f-b773-45d1-af83-1cd1570c2804/b948d429-f108-462e-8f18-75ba0a87c593"
-					(reference "Q19")
-					(unit 1)
-				)
 			)
 		)
@@
 					(unit 1)
 				)
-				(path "/b6fd875d-6e05-4440-9a05-0f0aa046a0ef/e121e58f-b773-45d1-af83-1cd1570c2804/b948d429-f108-462e-8f18-75ba0a87c593"
-					(reference "#PWR010")
-					(unit 1)
-				)
 			)
 		)
@@
 					(unit 1)
 				)
-				(path "/b6fd875d-6e05-4440-9a05-0f0aa046a0ef/e121e58f-b773-45d1-af83-1cd1570c2804/b948d429-f108-462e-8f18-75ba0a87c593"
-					(reference "Q20")
-					(unit 1)
-				)
 			)
 		)
@@
 					(unit 1)
 				)
-				(path "/b6fd875d-6e05-4440-9a05-0f0aa046a0ef/e121e58f-b773-45d1-af83-1cd1570c2804/b948d429-f108-462e-8f18-75ba0a87c593"
-					(reference "R84")
-					(unit 1)
-				)
 			)
 		)
@@
 					(unit 1)
 				)
-				(path "/b6fd875d-6e05-4440-9a05-0f0aa046a0ef/e121e58f-b773-45d1-af83-1cd1570c2804/b948d429-f108-462e-8f18-75ba0a87c593"
-					(reference "Q22")
-					(unit 1)
-				)
 			)
 		)
@@
 				(path "/b6fd875d-6e05-4440-9a05-0f0aa046a0ef/ad142cc2-d77f-4a6c-99c2-d9e17f4c27ae/8631bf3a-5019-45d5-a8fe-6e53ccedb3c2"
 					(reference "R63")
-					(unit 1)
-				)
-				(path "/b6fd875d-6e05-4440-9a05-0f0aa046a0ef/e121e58f-b773-45d1-af83-1cd1570c2804/b948d429-f108-462e-8f18-75ba0a87c593"
-					(reference "R82")
 					(unit 1)
 				)
@@
 					(unit 1)
 				)
-				(path "/b6fd875d-6e05-4440-9a05-0f0aa046a0ef/e121e58f-b773-45d1-af83-1cd1570c2804/b948d429-f108-462e-8f18-75ba0a87c593"
-					(reference "Q21")
-					(unit 1)
-				)
 			)
 		)
@@
 					(unit 1)
 				)
-				(path "/b6fd875d-6e05-4440-9a05-0f0aa046a0ef/e121e58f-b773-45d1-af83-1cd1570c2804/b948d429-f108-462e-8f18-75ba0a87c593"
-					(reference "R81")
-					(unit 1)
-				)
 			)
 		)
@@
 			)
 		)
-		(property "Value" "DNI (0R)"
+		(property "Value" "0R"
 			(at 144.78 139.446 90)
 			(effects
@@
 				(path "/b6fd875d-6e05-4440-9a05-0f0aa046a0ef/ad142cc2-d77f-4a6c-99c2-d9e17f4c27ae/8631bf3a-5019-45d5-a8fe-6e53ccedb3c2"
 					(reference "R71")
-					(unit 1)
-				)
-				(path "/b6fd875d-6e05-4440-9a05-0f0aa046a0ef/e121e58f-b773-45d1-af83-1cd1570c2804/b948d429-f108-462e-8f18-75ba0a87c593"
-					(reference "R90")
 					(unit 1)
 				)
@@
 					(unit 1)
 				)
-				(path "/b6fd875d-6e05-4440-9a05-0f0aa046a0ef/e121e58f-b773-45d1-af83-1cd1570c2804/b948d429-f108-462e-8f18-75ba0a87c593"
-					(reference "R83")
-					(unit 1)
-				)

Commit message: v3.1 Updates
Parts:
- C12: renamed from C14; value 10nF -> 10n
- C13: renamed from C15; value 10nF -> 10n
- R64: renamed from R71; now left out of the parts list
- R65: renamed from R72; now left out of the parts list
- renumbered Q16 to Q11, Q15 to Q12, Q18 to Q13, Q17 to Q14, R61 to R54, R62 to R55, R63 to R56, R64 to R57, R65 to R58, R66 to R59, R67 to R60, R68 to R61, R69 to R62, R70 to R63
Changed lines of the file:
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@@
 		(on_board yes)
 		(dnp no)
-		(property "Reference" "Q17"
-			(at 167.386 99.06 0)
+		(property "Reference" "Q14"
+			(at 167.64 99.06 0)
 			(effects
 				(font
@@
 			(project "BatteryBoard"
 				(path "/b6fd875d-6e05-4440-9a05-0f0aa046a0ef/ad142cc2-d77f-4a6c-99c2-d9e17f4c27ae/8631bf3a-5019-45d5-a8fe-6e53ccedb3c2"
-					(reference "Q17")
+					(reference "Q14")
 					(unit 2)
 				)
@@
 		(on_board yes)
 		(dnp no)
-		(property "Reference" "Q18"
+		(property "Reference" "Q13"
 			(at 172.72 72.009 90)
 			(effects
@@
 			(project "BatteryBoard"
 				(path "/b6fd875d-6e05-4440-9a05-0f0aa046a0ef/ad142cc2-d77f-4a6c-99c2-d9e17f4c27ae/8631bf3a-5019-45d5-a8fe-6e53ccedb3c2"
-					(reference "Q18")
+					(reference "Q13")
 					(unit 2)
 				)
@@
 		(unit 1)
 		(exclude_from_sim no)
-		(in_bom yes)
+		(in_bom no)
 		(on_board yes)
 		(dnp yes)
-		(property "Reference" "R72"
-			(at 144.78 142.621 90)
+		(property "Reference" "R65"
+			(at 144.78 142.494 90)
 			(effects
 				(font
@@
 		)
 		(property "Value" "0R"
-			(at 144.78 147.193 90)
+			(at 144.78 147.066 90)
 			(effects
 				(font
@@
 			(project "BatteryBoard"
 				(path "/b6fd875d-6e05-4440-9a05-0f0aa046a0ef/ad142cc2-d77f-4a6c-99c2-d9e17f4c27ae/8631bf3a-5019-45d5-a8fe-6e53ccedb3c2"
-					(reference "R72")
+					(reference "R65")
 					(unit 1)
 				)
@@
 		(on_board yes)
 		(dnp no)
-		(property "Reference" "Q16"
+		(property "Reference" "Q11"
 			(at 130.81 72.009 90)
 			(effects
@@
 			(project "BatteryBoard"
 				(path "/b6fd875d-6e05-4440-9a05-0f0aa046a0ef/ad142cc2-d77f-4a6c-99c2-d9e17f4c27ae/8631bf3a-5019-45d5-a8fe-6e53ccedb3c2"
-					(reference "Q16")
+					(reference "Q11")
 					(unit 2)
 				)
@@
 		(on_board yes)
 		(dnp no)
-		(property "Reference" "R70"
-			(at 178.816 91.694 0)
+		(property "Reference" "R63"
+			(at 179.07 91.694 0)
 			(effects
 				(font
@@
 		)
 		(property "Value" "200k"
-			(at 178.816 93.726 0)
+			(at 179.07 93.726 0)
 			(effects
 				(font
@@
 			(project "BatteryBoard"
 				(path "/b6fd875d-6e05-4440-9a05-0f0aa046a0ef/ad142cc2-d77f-4a6c-99c2-d9e17f4c27ae/8631bf3a-5019-45d5-a8fe-6e53ccedb3c2"
-					(reference "R70")
+					(reference "R63")
 					(unit 1)
 				)
@@
 		(on_board yes)
 		(dnp no)
-		(property "Reference" "R66"
-			(at 171.704 56.134 0)
+		(property "Reference" "R59"
+			(at 171.45 56.134 0)
 			(effects
 				(font
@@
 		)
 		(property "Value" "10k"
-			(at 171.704 58.166 0)
+			(at 171.45 58.166 0)
 			(effects
 				(font
@@
 			(project "BatteryBoard"
 				(path "/b6fd875d-6e05-4440-9a05-0f0aa046a0ef/ad142cc2-d77f-4a6c-99c2-d9e17f4c27ae/8631bf3a-5019-45d5-a8fe-6e53ccedb3c2"
-					(reference "R66")
+					(reference "R59")
 					(unit 1)
 				)
@@
 		(on_board yes)
 		(dnp no)
-		(property "Reference" "R61"
-			(at 129.667 56.134 0)
+		(property "Reference" "R54"
+			(at 129.54 56.134 0)
 			(effects
 				(font
@@
 			(project "BatteryBoard"
 				(path "/b6fd875d-6e05-4440-9a05-0f0aa046a0ef/ad142cc2-d77f-4a6c-99c2-d9e17f4c27ae/8631bf3a-5019-45d5-a8fe-6e53ccedb3c2"
-					(reference "R61")
+					(reference "R54")
 					(unit 1)
 				)
@@
 		(on_board yes)
 		(dnp no)
-		(property "Reference" "R68"
+		(property "Reference" "R61"
 			(at 161.29 74.676 90)
 			(effects
@@
 			(project "BatteryBoard"
 				(path "/b6fd875d-6e05-4440-9a05-0f0aa046a0ef/ad142cc2-d77f-4a6c-99c2-d9e17f4c27ae/8631bf3a-5019-45d5-a8fe-6e53ccedb3c2"
-					(reference "R68")
+					(reference "R61")
 					(unit 1)
 				)
@@
 		(on_board yes)
 		(dnp no)
-		(property "Reference" "C15"
-			(at 180.594 101.854 0)
-			(effects
-				(font
-					(size 1.27 1.27)
-				)
-				(justify left)
-			)
-		)
-		(property "Value" "10nF"
-			(at 180.594 103.886 0)
+		(property "Reference" "C13"
+			(at 180.34 101.854 0)
+			(effects
+				(font
+					(size 1.27 1.27)
+				)
+				(justify left)
+			)
+		)
+		(property "Value" "10n"
+			(at 180.34 103.886 0)
 			(effects
 				(font
@@
 			(project "BatteryBoard"
 				(path "/b6fd875d-6e05-4440-9a05-0f0aa046a0ef/ad142cc2-d77f-4a6c-99c2-d9e17f4c27ae/8631bf3a-5019-45d5-a8fe-6e53ccedb3c2"
-					(reference "C15")
+					(reference "C13")
 					(unit 1)
 				)
@@
 		(on_board yes)
 		(dnp no)
-		(property "Reference" "Q15"
-			(at 125.984 99.06 0)
+		(property "Reference" "Q12"
+			(at 125.73 99.06 0)
 			(effects
 				(font
@@
 			(project "BatteryBoard"
 				(path "/b6fd875d-6e05-4440-9a05-0f0aa046a0ef/ad142cc2-d77f-4a6c-99c2-d9e17f4c27ae/8631bf3a-5019-45d5-a8fe-6e53ccedb3c2"
-					(reference "Q15")
+					(reference "Q12")
 					(unit 2)
 				)
@@
 		(on_board yes)
 		(dnp no)
-		(property "Reference" "R69"
-			(at 163.576 89.154 0)
+		(property "Reference" "R62"
+			(at 163.83 89.154 0)
 			(effects
 				(font
@@
 		)
 		(property "Value" "100k"
-			(at 163.576 90.932 0)
+			(at 163.83 91.186 0)
 			(effects
 				(font
@@
 			(project "BatteryBoard"
 				(path "/b6fd875d-6e05-4440-9a05-0f0aa046a0ef/ad142cc2-d77f-4a6c-99c2-d9e17f4c27ae/8631bf3a-5019-45d5-a8fe-6e53ccedb3c2"
-					(reference "R69")
+					(reference "R62")
 					(unit 1)
 				)
@@
 		(on_board yes)
 		(dnp no)
-		(property "Reference" "R67"
-			(at 178.816 62.484 0)
+		(property "Reference" "R60"
+			(at 179.07 62.484 0)
 			(effects
 				(font
@@
 		)
 		(property "Value" "10k"
-			(at 178.816 64.516 0)
+			(at 179.07 64.516 0)
 			(effects
 				(font
@@
 			(project "BatteryBoard"
 				(path "/b6fd875d-6e05-4440-9a05-0f0aa046a0ef/ad142cc2-d77f-4a6c-99c2-d9e17f4c27ae/8631bf3a-5019-45d5-a8fe-6e53ccedb3c2"
-					(reference "R67")
+					(reference "R60")
 					(unit 1)
 				)
@@
 		(on_board yes)
 		(dnp no)
-		(property "Reference" "C14"
-			(at 138.684 101.854 0)
-			(effects
-				(font
-					(size 1.27 1.27)
-				)
-				(justify left)
-			)
-		)
-		(property "Value" "10nF"
-			(at 138.684 103.9114 0)
+		(property "Reference" "C12"
+			(at 138.43 101.854 0)
+			(effects
+				(font
+					(size 1.27 1.27)
+				)
+				(justify left)
+			)
+		)
+		(property "Value" "10n"
+			(at 138.43 103.886 0)
 			(effects
 				(font
@@
 			(project "BatteryBoard"
 				(path "/b6fd875d-6e05-4440-9a05-0f0aa046a0ef/ad142cc2-d77f-4a6c-99c2-d9e17f4c27ae/8631bf3a-5019-45d5-a8fe-6e53ccedb3c2"
-					(reference "C14")
+					(reference "C12")
 					(unit 1)
 				)
@@
 		(on_board yes)
 		(dnp no)
-		(property "Reference" "Q15"
+		(property "Reference" "Q12"
 			(at 110.49 93.98 0)
 			(effects
@@
 			(project "BatteryBoard"
 				(path "/b6fd875d-6e05-4440-9a05-0f0aa046a0ef/ad142cc2-d77f-4a6c-99c2-d9e17f4c27ae/8631bf3a-5019-45d5-a8fe-6e53ccedb3c2"
-					(reference "Q15")
+					(reference "Q12")
 					(unit 1)
 				)
@@
 		(on_board yes)
 		(dnp no)
-		(property "Reference" "Q16"
+		(property "Reference" "Q11"
 			(at 130.81 89.408 90)
 			(effects
@@
 			(project "BatteryBoard"
 				(path "/b6fd875d-6e05-4440-9a05-0f0aa046a0ef/ad142cc2-d77f-4a6c-99c2-d9e17f4c27ae/8631bf3a-5019-45d5-a8fe-6e53ccedb3c2"
-					(reference "Q16")
+					(reference "Q11")
 					(unit 1)
 				)
@@
 		(on_board yes)
 		(dnp no)
-		(property "Reference" "R65"
-			(at 137.033 91.694 0)
+		(property "Reference" "R58"
+			(at 137.16 91.694 0)
 			(effects
 				(font
@@
 		)
 		(property "Value" "200k"
-			(at 137.033 93.726 0)
+			(at 137.16 93.726 0)
 			(effects
 				(font
@@
 			(project "BatteryBoard"
 				(path "/b6fd875d-6e05-4440-9a05-0f0aa046a0ef/ad142cc2-d77f-4a6c-99c2-d9e17f4c27ae/8631bf3a-5019-45d5-a8fe-6e53ccedb3c2"
-					(reference "R65")
+					(reference "R58")
 					(unit 1)
 				)
@@
 		(on_board yes)
 		(dnp no)
-		(property "Reference" "Q18"
+		(property "Reference" "Q13"
 			(at 172.72 89.408 90)
 			(effects
@@
 			(project "BatteryBoard"
 				(path "/b6fd875d-6e05-4440-9a05-0f0aa046a0ef/ad142cc2-d77f-4a6c-99c2-d9e17f4c27ae/8631bf3a-5019-45d5-a8fe-6e53ccedb3c2"
-					(reference "Q18")
+					(reference "Q13")
 					(unit 1)
 				)
@@
 		(on_board yes)
 		(dnp no)
-		(property "Reference" "R63"
+		(property "Reference" "R56"
 			(at 119.38 74.676 90)
 			(effects
@@
 			(project "BatteryBoard"
 				(path "/b6fd875d-6e05-4440-9a05-0f0aa046a0ef/ad142cc2-d77f-4a6c-99c2-d9e17f4c27ae/8631bf3a-5019-45d5-a8fe-6e53ccedb3c2"
-					(reference "R63")
+					(reference "R56")
 					(unit 1)
 				)
@@
 		(on_board yes)
 		(dnp no)
-		(property "Reference" "Q17"
+		(property "Reference" "Q14"
 			(at 152.4 93.98 0)
 			(effects
@@
 			(project "BatteryBoard"
 				(path "/b6fd875d-6e05-4440-9a05-0f0aa046a0ef/ad142cc2-d77f-4a6c-99c2-d9e17f4c27ae/8631bf3a-5019-45d5-a8fe-6e53ccedb3c2"
-					(reference "Q17")
+					(reference "Q14")
 					(unit 1)
 				)
@@
 		(on_board yes)
 		(dnp no)
-		(property "Reference" "R62"
-			(at 137.033 62.484 0)
+		(property "Reference" "R55"
+			(at 137.16 62.484 0)
 			(effects
 				(font
@@
 		)
 		(property "Value" "10k"
-			(at 137.033 64.516 0)
+			(at 137.16 64.516 0)
 			(effects
 				(font
@@
 			(project "BatteryBoard"
 				(path "/b6fd875d-6e05-4440-9a05-0f0aa046a0ef/ad142cc2-d77f-4a6c-99c2-d9e17f4c27ae/8631bf3a-5019-45d5-a8fe-6e53ccedb3c2"
-					(reference "R62")
+					(reference "R55")
 					(unit 1)
 				)
@@
 		(unit 1)
 		(exclude_from_sim no)
-		(in_bom yes)
+		(in_bom no)
 		(on_board yes)
 		(dnp yes)
-		(property "Reference" "R71"
+		(property "Reference" "R64"
 			(at 144.78 134.874 90)
 			(effects
@@
 			(project "BatteryBoard"
 				(path "/b6fd875d-6e05-4440-9a05-0f0aa046a0ef/ad142cc2-d77f-4a6c-99c2-d9e17f4c27ae/8631bf3a-5019-45d5-a8fe-6e53ccedb3c2"
-					(reference "R71")
+					(reference "R64")
 					(unit 1)
 				)
@@
 		(on_board yes)
 		(dnp no)
-		(property "Reference" "R64"
-			(at 121.793 89.154 0)
+		(property "Reference" "R57"
+			(at 121.92 89.154 0)
 			(effects
 				(font
@@
 		)
 		(property "Value" "100k"
-			(at 121.793 91.186 0)
+			(at 121.92 91.186 0)
 			(effects
 				(font
@@
 			(project "BatteryBoard"
 				(path "/b6fd875d-6e05-4440-9a05-0f0aa046a0ef/ad142cc2-d77f-4a6c-99c2-d9e17f4c27ae/8631bf3a-5019-45d5-a8fe-6e53ccedb3c2"
-					(reference "R64")
-					(unit 1)
-				)
+					(reference "R57")
+					(unit 1)
+				)
