File: I2CProtection.kicad_sch (KiCad schematic)
At the start: 18 parts, among them Q11 MBT2222ADW1T1, Q12 NX3008NBKS, Q13 MBT2222ADW1T1, Q14 NX3008NBKS

Commit message: Idk some changes
Parts:
- C12, C13: MPN (none) -> C161232
- Q12, Q14: MPN (none) -> C3280240; Manufacturer_Name Nexperia USA Inc. -> (none); Manufacturer_Part_Number NX3008NBKS -> (none); Proto BSS138DWQ-7 -> (none)
- R54, R55, R59, R60: MPN (none) -> C2479067
- R56, R61: MPN (none) -> C844802
- R57, R62: MPN (none) -> C237792
- R58, R63: MPN (none) -> C118142
Other:
- moved on the sheet: C12, C13

Commit message: Local Stash
Parts:
- Q12, Q14: symbol Device:Q_Dual_NMOS_S1G1D2S2G2D1 -> Argus-IC:Q_Dual_NMOS_S1G1D2S2G2D1
Changed lines of the file:
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@@
 	(title_block
 		(title "Argus Batteryboard")
-		(date "2025-01-08")
-		(rev "v3.0")
+		(date "2025-04-16")
+		(rev "v3.1")
 		(company "Carnegie Mellon University")
 		(comment 1 "M. Holliday")
@@
 	)
 	(symbol
-		(lib_id "Device:Q_Dual_NMOS_S1G1D2S2G2D1")
+		(lib_id "Argus-IC:Q_Dual_NMOS_S1G1D2S2G2D1")
 		(at 172.72 99.06 0)
 		(mirror y)
@@
 	)
 	(symbol
-		(lib_id "Device:Q_Dual_NMOS_S1G1D2S2G2D1")
+		(lib_id "Argus-IC:Q_Dual_NMOS_S1G1D2S2G2D1")
 		(at 130.81 99.06 0)
 		(mirror y)
@@
 	)
 	(symbol
-		(lib_id "Device:Q_Dual_NMOS_S1G1D2S2G2D1")
+		(lib_id "Argus-IC:Q_Dual_NMOS_S1G1D2S2G2D1")
 		(at 115.57 93.98 0)
 		(mirror y)
@@
 	)
 	(symbol
-		(lib_id "Device:Q_Dual_NMOS_S1G1D2S2G2D1")
+		(lib_id "Argus-IC:Q_Dual_NMOS_S1G1D2S2G2D1")
 		(at 157.48 93.98 0)
 		(mirror y)
