File: I2CProtection.kicad_sch (KiCad schematic)
At the start: 18 parts, among them Q11 MBT2222ADW1T1, Q12 NX3008NBKS, Q13 MBT2222ADW1T1, Q14 NX3008NBKS

Commit message: making a few changes
Other:
- title: Argus Batteryboard -> Batteryboard
Changed lines of the file:
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@@
 	(paper "A4")
 	(title_block
-		(title "Argus Batteryboard")
-		(date "2026-04-14")
-		(rev "v3.2")
+		(title "Batteryboard")
+		(date "2026-08-21")
+		(rev "v4.0")
 		(company "Carnegie Mellon University")
-		(comment 1 "M. Holliday")
-		(comment 2 "N. Khera")
-		(comment 3 "V. Rajesh")
+		(comment 1 "N. Khera")
+		(comment 2 "V. Rajesh")
+		(comment 3 "S. Farhan")
 	)
 	(text "I2C Bus Protection"

Commit message: routing
Parts:
- renumbered Q11 to Q5, Q13 to Q6, Q12 to Q7, Q14 to Q8, R54 to R26, R59 to R27, R55 to R28, R60 to R29, R56 to R30, R61 to R31, R57 to R32, R62 to R33, R58 to R34, R63 to R35, R64 to R36, R65 to R37
Changed lines of the file:
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@@
 		(in_pos_files yes)
 		(dnp no)
-		(property "Reference" "Q14"
+		(property "Reference" "Q8"
 			(at 167.64 99.06 0)
 			(show_name no)
@@
 			(project "Avionics-BatteryBoard"
 				(path "/b6fd875d-6e05-4440-9a05-0f0aa046a0ef/ad142cc2-d77f-4a6c-99c2-d9e17f4c27ae/8631bf3a-5019-45d5-a8fe-6e53ccedb3c2"
-					(reference "Q14")
+					(reference "Q8")
 					(unit 2)
 				)
@@
 		(in_pos_files yes)
 		(dnp no)
-		(property "Reference" "Q13"
+		(property "Reference" "Q6"
 			(at 172.72 72.009 90)
 			(show_name no)
@@
 			(project "Avionics-BatteryBoard"
 				(path "/b6fd875d-6e05-4440-9a05-0f0aa046a0ef/ad142cc2-d77f-4a6c-99c2-d9e17f4c27ae/8631bf3a-5019-45d5-a8fe-6e53ccedb3c2"
-					(reference "Q13")
+					(reference "Q6")
 					(unit 2)
 				)
@@
 		(in_pos_files yes)
 		(dnp no)
-		(property "Reference" "#PWR08"
+		(property "Reference" "#PWR019"
 			(at 177.8 116.84 0)
 			(hide yes)
@@
 			(project "Avionics-BatteryBoard"
 				(path "/b6fd875d-6e05-4440-9a05-0f0aa046a0ef/ad142cc2-d77f-4a6c-99c2-d9e17f4c27ae/8631bf3a-5019-45d5-a8fe-6e53ccedb3c2"
-					(reference "#PWR08")
+					(reference "#PWR019")
 					(unit 1)
 				)
@@
 		(in_pos_files yes)
 		(dnp no)
-		(property "Reference" "#PWR06"
+		(property "Reference" "#PWR017"
 			(at 162.56 90.17 0)
 			(hide yes)
@@
 			(project "Avionics-BatteryBoard"
 				(path "/b6fd875d-6e05-4440-9a05-0f0aa046a0ef/ad142cc2-d77f-4a6c-99c2-d9e17f4c27ae/8631bf3a-5019-45d5-a8fe-6e53ccedb3c2"
-					(reference "#PWR06")
+					(reference "#PWR017")
 					(unit 1)
 				)
@@
 		(in_pos_files yes)
 		(dnp yes)
-		(property "Reference" "R65"
+		(property "Reference" "R37"
 			(at 144.78 142.494 90)
 			(show_name no)
@@
 			(project "Avionics-BatteryBoard"
 				(path "/b6fd875d-6e05-4440-9a05-0f0aa046a0ef/ad142cc2-d77f-4a6c-99c2-d9e17f4c27ae/8631bf3a-5019-45d5-a8fe-6e53ccedb3c2"
-					(reference "R65")
+					(reference "R37")
 					(unit 1)
 				)
@@
 		(in_pos_files yes)
 		(dnp no)
-		(property "Reference" "#PWR02"
+		(property "Reference" "#PWR016"
 			(at 120.65 90.17 0)
 			(hide yes)
@@
 			(project "Avionics-BatteryBoard"
 				(path "/b6fd875d-6e05-4440-9a05-0f0aa046a0ef/ad142cc2-d77f-4a6c-99c2-d9e17f4c27ae/8631bf3a-5019-45d5-a8fe-6e53ccedb3c2"
-					(reference "#PWR02")
+					(reference "#PWR016")
 					(unit 1)
 				)
@@
 		(in_pos_files yes)
 		(dnp no)
-		(property "Reference" "Q11"
+		(property "Reference" "Q5"
 			(at 130.81 72.009 90)
 			(show_name no)
@@
 			(project "Avionics-BatteryBoard"
 				(path "/b6fd875d-6e05-4440-9a05-0f0aa046a0ef/ad142cc2-d77f-4a6c-99c2-d9e17f4c27ae/8631bf3a-5019-45d5-a8fe-6e53ccedb3c2"
-					(reference "Q11")
+					(reference "Q5")
 					(unit 2)
 				)
@@
 		(in_pos_files yes)
 		(dnp no)
-		(property "Reference" "R63"
+		(property "Reference" "R35"
 			(at 179.07 91.694 0)
 			(show_name no)
@@
 			(project "Avionics-BatteryBoard"
 				(path "/b6fd875d-6e05-4440-9a05-0f0aa046a0ef/ad142cc2-d77f-4a6c-99c2-d9e17f4c27ae/8631bf3a-5019-45d5-a8fe-6e53ccedb3c2"
-					(reference "R63")
+					(reference "R35")
 					(unit 1)
 				)
@@
 		(in_pos_files yes)
 		(dnp no)
-		(property "Reference" "R59"
+		(property "Reference" "R27"
 			(at 171.45 56.134 0)
 			(show_name no)
@@
 			(project "Avionics-BatteryBoard"
 				(path "/b6fd875d-6e05-4440-9a05-0f0aa046a0ef/ad142cc2-d77f-4a6c-99c2-d9e17f4c27ae/8631bf3a-5019-45d5-a8fe-6e53ccedb3c2"
-					(reference "R59")
+					(reference "R27")
 					(unit 1)
 				)
@@
 		(in_pos_files yes)
 		(dnp no)
-		(property "Reference" "R54"
+		(property "Reference" "R26"
 			(at 129.54 56.134 0)
 			(show_name no)
@@
 			(project "Avionics-BatteryBoard"
 				(path "/b6fd875d-6e05-4440-9a05-0f0aa046a0ef/ad142cc2-d77f-4a6c-99c2-d9e17f4c27ae/8631bf3a-5019-45d5-a8fe-6e53ccedb3c2"
-					(reference "R54")
+					(reference "R26")
 					(unit 1)
 				)
@@
 		(in_pos_files yes)
 		(dnp no)
-		(property "Reference" "R61"
+		(property "Reference" "R31"
 			(at 161.29 74.676 90)
 			(show_name no)
@@
 			(project "Avionics-BatteryBoard"
 				(path "/b6fd875d-6e05-4440-9a05-0f0aa046a0ef/ad142cc2-d77f-4a6c-99c2-d9e17f4c27ae/8631bf3a-5019-45d5-a8fe-6e53ccedb3c2"
-					(reference "R61")
+					(reference "R31")
 					(unit 1)
 				)
@@
 		(in_pos_files yes)
 		(dnp no)
-		(property "Reference" "#PWR07"
+		(property "Reference" "#PWR015"
 			(at 172.72 55.88 0)
 			(hide yes)
@@
 			(project "Avionics-BatteryBoard"
 				(path "/b6fd875d-6e05-4440-9a05-0f0aa046a0ef/ad142cc2-d77f-4a6c-99c2-d9e17f4c27ae/8631bf3a-5019-45d5-a8fe-6e53ccedb3c2"
-					(reference "#PWR07")
+					(reference "#PWR015")
 					(unit 1)
 				)
@@
 		(in_pos_files yes)
 		(dnp no)
-		(property "Reference" "#PWR05"
+		(property "Reference" "#PWR018"
 			(at 135.89 116.84 0)
 			(hide yes)
@@
 			(project "Avionics-BatteryBoard"
 				(path "/b6fd875d-6e05-4440-9a05-0f0aa046a0ef/ad142cc2-d77f-4a6c-99c2-d9e17f4c27ae/8631bf3a-5019-45d5-a8fe-6e53ccedb3c2"
-					(reference "#PWR05")
+					(reference "#PWR018")
 					(unit 1)
 				)
@@
 		(in_pos_files yes)
 		(dnp no)
-		(property "Reference" "Q12"
+		(property "Reference" "Q7"
 			(at 125.73 99.06 0)
 			(show_name no)
@@
 			(project "Avionics-BatteryBoard"
 				(path "/b6fd875d-6e05-4440-9a05-0f0aa046a0ef/ad142cc2-d77f-4a6c-99c2-d9e17f4c27ae/8631bf3a-5019-45d5-a8fe-6e53ccedb3c2"
-					(reference "Q12")
+					(reference "Q7")
 					(unit 2)
 				)
@@
 		(in_pos_files yes)
 		(dnp no)
-		(property "Reference" "R62"
+		(property "Reference" "R33"
 			(at 163.83 89.154 0)
 			(show_name no)
@@
 			(project "Avionics-BatteryBoard"
 				(path "/b6fd875d-6e05-4440-9a05-0f0aa046a0ef/ad142cc2-d77f-4a6c-99c2-d9e17f4c27ae/8631bf3a-5019-45d5-a8fe-6e53ccedb3c2"
-					(reference "R62")
+					(reference "R33")
 					(unit 1)
 				)
@@
 		(in_pos_files yes)
 		(dnp no)
-		(property "Reference" "R60"
+		(property "Reference" "R29"
 			(at 179.07 62.484 0)
 			(show_name no)
@@
 			(project "Avionics-BatteryBoard"
 				(path "/b6fd875d-6e05-4440-9a05-0f0aa046a0ef/ad142cc2-d77f-4a6c-99c2-d9e17f4c27ae/8631bf3a-5019-45d5-a8fe-6e53ccedb3c2"
-					(reference "R60")
+					(reference "R29")
 					(unit 1)
 				)
@@
 		(in_pos_files yes)
 		(dnp no)
-		(property "Reference" "Q12"
+		(property "Reference" "Q7"
 			(at 110.49 93.98 0)
 			(show_name no)
@@
 			(project "Avionics-BatteryBoard"
 				(path "/b6fd875d-6e05-4440-9a05-0f0aa046a0ef/ad142cc2-d77f-4a6c-99c2-d9e17f4c27ae/8631bf3a-5019-45d5-a8fe-6e53ccedb3c2"
-					(reference "Q12")
+					(reference "Q7")
 					(unit 1)
 				)
@@
 		(in_pos_files yes)
 		(dnp no)
-		(property "Reference" "#PWR04"
+		(property "Reference" "#PWR014"
 			(at 130.81 55.88 0)
 			(hide yes)
@@
 			(project "Avionics-BatteryBoard"
 				(path "/b6fd875d-6e05-4440-9a05-0f0aa046a0ef/ad142cc2-d77f-4a6c-99c2-d9e17f4c27ae/8631bf3a-5019-45d5-a8fe-6e53ccedb3c2"
-					(reference "#PWR04")
+					(reference "#PWR014")
 					(unit 1)
 				)
@@
 		(in_pos_files yes)
 		(dnp no)
-		(property "Reference" "Q11"
+		(property "Reference" "Q5"
 			(at 130.81 89.408 90)
 			(show_name no)
@@
 			(project "Avionics-BatteryBoard"
 				(path "/b6fd875d-6e05-4440-9a05-0f0aa046a0ef/ad142cc2-d77f-4a6c-99c2-d9e17f4c27ae/8631bf3a-5019-45d5-a8fe-6e53ccedb3c2"
-					(reference "Q11")
+					(reference "Q5")
 					(unit 1)
 				)
@@
 		(in_pos_files yes)
 		(dnp no)
-		(property "Reference" "R58"
+		(property "Reference" "R34"
 			(at 137.16 91.694 0)
 			(show_name no)
@@
 			(project "Avionics-BatteryBoard"
 				(path "/b6fd875d-6e05-4440-9a05-0f0aa046a0ef/ad142cc2-d77f-4a6c-99c2-d9e17f4c27ae/8631bf3a-5019-45d5-a8fe-6e53ccedb3c2"
-					(reference "R58")
+					(reference "R34")
 					(unit 1)
 				)
@@
 		(in_pos_files yes)
 		(dnp no)
-		(property "Reference" "Q13"
+		(property "Reference" "Q6"
 			(at 172.72 89.408 90)
 			(show_name no)
@@
 			(project "Avionics-BatteryBoard"
 				(path "/b6fd875d-6e05-4440-9a05-0f0aa046a0ef/ad142cc2-d77f-4a6c-99c2-d9e17f4c27ae/8631bf3a-5019-45d5-a8fe-6e53ccedb3c2"
-					(reference "Q13")
+					(reference "Q6")
 					(unit 1)
 				)
@@
 		(in_pos_files yes)
 		(dnp no)
-		(property "Reference" "R56"
+		(property "Reference" "R30"
 			(at 119.38 74.676 90)
 			(show_name no)
@@
 			(project "Avionics-BatteryBoard"
 				(path "/b6fd875d-6e05-4440-9a05-0f0aa046a0ef/ad142cc2-d77f-4a6c-99c2-d9e17f4c27ae/8631bf3a-5019-45d5-a8fe-6e53ccedb3c2"
-					(reference "R56")
+					(reference "R30")
 					(unit 1)
 				)
@@
 		(in_pos_files yes)
 		(dnp no)
-		(property "Reference" "Q14"
+		(property "Reference" "Q8"
 			(at 152.4 93.98 0)
 			(show_name no)
@@
 			(project "Avionics-BatteryBoard"
 				(path "/b6fd875d-6e05-4440-9a05-0f0aa046a0ef/ad142cc2-d77f-4a6c-99c2-d9e17f4c27ae/8631bf3a-5019-45d5-a8fe-6e53ccedb3c2"
-					(reference "Q14")
+					(reference "Q8")
 					(unit 1)
 				)
@@
 		(in_pos_files yes)
 		(dnp no)
-		(property "Reference" "R55"
+		(property "Reference" "R28"
 			(at 137.16 62.484 0)
 			(show_name no)
@@
 			(project "Avionics-BatteryBoard"
 				(path "/b6fd875d-6e05-4440-9a05-0f0aa046a0ef/ad142cc2-d77f-4a6c-99c2-d9e17f4c27ae/8631bf3a-5019-45d5-a8fe-6e53ccedb3c2"
-					(reference "R55")
+					(reference "R28")
 					(unit 1)
 				)
@@
 		(in_pos_files yes)
 		(dnp yes)
-		(property "Reference" "R64"
+		(property "Reference" "R36"
 			(at 144.78 134.874 90)
 			(show_name no)
@@
 			(project "Avionics-BatteryBoard"
 				(path "/b6fd875d-6e05-4440-9a05-0f0aa046a0ef/ad142cc2-d77f-4a6c-99c2-d9e17f4c27ae/8631bf3a-5019-45d5-a8fe-6e53ccedb3c2"
-					(reference "R64")
+					(reference "R36")
 					(unit 1)
 				)
@@
 		(in_pos_files yes)
 		(dnp no)
-		(property "Reference" "R57"
+		(property "Reference" "R32"
 			(at 121.92 89.154 0)
 			(show_name no)
@@
 			(project "Avionics-BatteryBoard"
 				(path "/b6fd875d-6e05-4440-9a05-0f0aa046a0ef/ad142cc2-d77f-4a6c-99c2-d9e17f4c27ae/8631bf3a-5019-45d5-a8fe-6e53ccedb3c2"
-					(reference "R57")
+					(reference "R32")
 					(unit 1)
 				)
