File: Battery.kicad_sch (KiCad schematic)
At the start: 12 parts, among them J1 Keystone-1048, J5 Keystone-1042, J6 Keystone-1042, J9 Keystone-1048

Commit message: Changes for lib refactor
Parts:
- J1, J9: footprint Battery-Board:BAT_1048 -> Argus-Misc:BAT_1048; symbol Battery-Board:Keystone-1048 -> Argus-Misc:Keystone-1048
- J5, J6: footprint Battery-Board:Keystone_1042 -> Argus-Misc:Keystone_1042; symbol Battery-Board:Keystone-1042 -> Argus-Misc:Keystone-1042
Changed lines of the file:
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@@
 	)
 	(symbol
-		(lib_id "Battery-Board:Keystone-1042")
+		(lib_id "Argus-Misc:Keystone-1042")
 		(at 133.35 107.95 90)
 		(unit 1)
@@
 			)
 		)
-		(property "Footprint" "Battery-Board:Keystone_1042"
+		(property "Footprint" "Argus-Misc:Keystone_1042"
 			(at 133.35 107.95 0)
 			(effects
@@
 	)
 	(symbol
-		(lib_id "Battery-Board:Keystone-1042")
+		(lib_id "Argus-Misc:Keystone-1042")
 		(at 133.35 80.01 90)
 		(unit 1)
@@
 			)
 		)
-		(property "Footprint" "Battery-Board:Keystone_1042"
+		(property "Footprint" "Argus-Misc:Keystone_1042"
 			(at 133.35 80.01 0)
 			(effects
@@
 	)
 	(symbol
-		(lib_id "Battery-Board:Keystone-1048")
+		(lib_id "Argus-Misc:Keystone-1048")
 		(at 115.57 109.22 90)
 		(unit 1)
@@
 			)
 		)
-		(property "Footprint" "Battery-Board:BAT_1048"
+		(property "Footprint" "Argus-Misc:BAT_1048"
 			(at 124.714 109.22 0)
 			(effects
@@
 	)
 	(symbol
-		(lib_id "Battery-Board:Keystone-1048")
+		(lib_id "Argus-Misc:Keystone-1048")
 		(at 115.57 80.01 90)
 		(unit 1)
@@
 			)
 		)
-		(property "Footprint" "Battery-Board:BAT_1048"
+		(property "Footprint" "Argus-Misc:BAT_1048"
 			(at 124.714 80.01 0)
 			(effects

Commit message: v2.1 (v3?) Partial Updates
Parts:
- D1: renamed from D7; symbol Device:D_Schottky -> Device:D_Schottky_Small
- D2: renamed from D6; symbol Device:D_Schottky -> Device:D_Schottky_Small
- renumbered F12 to F1, F10 to F2, F9 to F3, F7 to F4, F6 to F5, F4 to F6, J9 to J2, J6 to J3, J5 to J4
Connections:
- net BATT0 renamed BATT_N
- net BATT1 renamed BATT_M
- net BATT2 renamed BATT_P
Other:
- note added: "6x 18650 cells in 2S3P arrangement Panasonic NCR18650GA. 3450mAh. 10350mAh total Samsung 35E. 3500mAh = 10500mAh total 7.2V nominal, 8.4V max"
- note added: "Must install low-side before high-side"
- company: (none) -> Carnegie Mellon University
- title: (none) -> Argus Batteryboard
- moved on the sheet: D1, D2, F1, F2, F3, F4, F5, F6, J1, J2, J3, J4

Commit message: Finalized updates with recommendations and exported files
Parts:
- D1, D2: value 10V Vrm -> BAT60JFILM; footprint Diode_SMD:D_SOD-123F -> Diode_SMD:D_SOD-323_HandSoldering; Field5 (none) -> 10V Vrm
- F1, F2, F3, F4, F5, F6: value 10A -> 5A
Connections:
- net BATT_N: now also F1.2, F3.2
- net BATT_P: now also F2.2, F4.2
- net at F5.1, J3.1 (NEG): no longer F3.2
- net at F3.1, J1.3 (NEG): no longer F1.2
- net at F4.1, J2.4 (POS): no longer F2.2
- net at F6.1, J4.2 (POS): no longer F4.2
Other:
- moved on the sheet: D1, D2, F1, F2, F3, F4, F5, F6, J3, J4

Commit message: v3.1 Updates
Parts:
- D1, D2: Flight (none) -> DNI
- F1, F2, F3, F4, F5, F6: Flight (none) -> 0R
Changed lines of the file:
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@@
+			)
+		)
+		(property "Flight" "0R"
+			(at 109.22 108.458 0)
+			(effects
+				(font
+					(size 1.27 1.27)
+				)
 			)
 		)
@@
 			)
 		)
+		(property "Flight" "DNI"
+			(at 124.46 127.508 0)
+			(effects
+				(font
+					(size 1.27 1.27)
+				)
+			)
+		)
 		(pin "1"
 		)
@@
 		(dnp no)
 		(property "Reference" "F3"
-			(at 107.95 91.44 0)
-			(effects
-				(font
-					(size 1.27 1.27)
-				)
-				(justify right)
+			(at 109.22 91.44 0)
+			(effects
+				(font
+					(size 1.27 1.27)
+				)
 			)
 		)
@@
 			)
 		)
+		(property "Flight" "0R"
+			(at 109.22 97.028 0)
+			(effects
+				(font
+					(size 1.27 1.27)
+				)
+			)
+		)
 		(pin "2"
 		)
@@
 			)
 		)
+		(property "Flight" "0R"
+			(at 167.64 86.868 0)
+			(effects
+				(font
+					(size 1.27 1.27)
+				)
+			)
+		)
 		(pin "2"
 		)
@@
 			)
 		)
+		(property "Flight" "0R"
+			(at 167.64 108.458 0)
+			(effects
+				(font
+					(size 1.27 1.27)
+				)
+			)
+		)
 		(pin "2"
 		)
@@
 			)
 		)
+		(property "Flight" "DNI"
+			(at 152.4 127.508 0)
+			(effects
+				(font
+					(size 1.27 1.27)
+				)
+			)
+		)
 		(pin "1"
 		)
@@
 			)
 		)
+		(property "Flight" "0R"
+			(at 109.22 86.868 0)
+			(effects
+				(font
+					(size 1.27 1.27)
+				)
+			)
+		)
 		(pin "2"
 		)
@@
 			)
 		)
+		(property "Flight" "0R"
+			(at 167.64 97.028 0)
+			(effects
+				(font
+					(size 1.27 1.27)
+				)
+			)
+		)

Commit message: Idk some changes
Parts:
- F1, F2, F3, F4, F5, F6: MPN (none) -> C844862
Changed lines of the file:
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@@
+			)
+		)
+		(property "MPN" "C844862"
+			(at 109.22 106.68 0)
+			(effects
+				(font
+					(size 1.27 1.27)
+				)
+				(hide yes)
 			)
 		)
@@
 			)
 		)
+		(property "MPN" "C844862"
+			(at 109.22 95.25 0)
+			(effects
+				(font
+					(size 1.27 1.27)
+				)
+				(hide yes)
+			)
+		)
 		(pin "2"
 		)
@@
 			)
 		)
+		(property "MPN" "C844862"
+			(at 167.64 85.09 0)
+			(effects
+				(font
+					(size 1.27 1.27)
+				)
+				(hide yes)
+			)
+		)
 		(pin "2"
 		)
@@
 			)
 		)
+		(property "MPN" "C844862"
+			(at 167.64 106.68 0)
+			(effects
+				(font
+					(size 1.27 1.27)
+				)
+				(hide yes)
+			)
+		)
 		(pin "2"
 		)
@@
 			)
 		)
+		(property "MPN" "C844862"
+			(at 109.22 85.09 0)
+			(effects
+				(font
+					(size 1.27 1.27)
+				)
+				(hide yes)
+			)
+		)
 		(pin "2"
 		)
@@
 			)
 		)
+		(property "MPN" "C844862"
+			(at 167.64 95.25 0)
+			(effects
+				(font
+					(size 1.27 1.27)
+				)
+				(hide yes)
+			)
+		)
