File: BatteryBusProtection.kicad_sch (KiCad schematic)
At the start: 14 parts, among them Q11 SIRA99DP-T1-GE3, Q12 SIRA99DP-T1-GE3, Q13 SIRA99DP-T1-GE3, Q14 SIRA99DP-T1-GE3, U4 LTC4412xS6, U5 LTC4412xS6

Commit message: v3.1 Updates
Parts:
- C5: renamed from C7; value 0.1uF -> 100n
- C6: renamed from C8; value 0.1uF -> 100n
- F7, F8: symbol Device:Fuse -> Device:Fuse_Small
- renumbered Q14 to Q10, Q11 to Q7, Q12 to Q8, Q13 to Q9, R44 to R37, R45 to R38, R46 to R39, R47 to R40, U4 to U3, U5 to U4
Other:
- moved on the sheet: F7, F8
Changed lines of the file:
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@@
 	(wire
 		(pts
-			(xy 100.33 45.72) (xy 109.22 45.72)
+			(xy 100.33 45.72) (xy 110.49 45.72)
 		)
 		(stroke
@@
 	(wire
 		(pts
+			(xy 115.57 110.49) (xy 124.46 110.49)
+		)
+		(stroke
+			(width 0)
+			(type default)
+		)
+	)
+	(wire
+		(pts
 			(xy 116.84 71.12) (xy 119.38 71.12)
 		)
@@
 	(wire
 		(pts
-			(xy 116.84 45.72) (xy 130.81 45.72)
-		)
-		(stroke
-			(width 0)
-			(type default)
-		)
-	)
-	(wire
-		(pts
 			(xy 124.46 110.49) (xy 124.46 118.11)
 		)
@@
 	(wire
 		(pts
-			(xy 100.33 110.49) (xy 109.22 110.49)
+			(xy 100.33 110.49) (xy 110.49 110.49)
 		)
 		(stroke
@@
 	(wire
 		(pts
-			(xy 116.84 110.49) (xy 124.46 110.49)
-		)
-		(stroke
-			(width 0)
-			(type default)
-		)
-	)
-	(wire
-		(pts
 			(xy 135.89 66.04) (xy 147.32 66.04)
 		)
@@
 		(pts
 			(xy 152.4 110.49) (xy 165.1 110.49)
+		)
+		(stroke
+			(width 0)
+			(type default)
+		)
+	)
+	(wire
+		(pts
+			(xy 115.57 45.72) (xy 130.81 45.72)
 		)
 		(stroke
@@
 		(on_board yes)
 		(dnp no)
-		(property "Reference" "R46"
-			(at 129.54 119.634 0)
-			(effects
-				(font
-					(size 1.27 1.27)
-				)
-				(justify left)
+		(property "Reference" "R39"
+			(at 125.73 119.634 0)
+			(effects
+				(font
+					(size 1.27 1.27)
+				)
+				(justify right)
 			)
 		)
 		(property "Value" "100k"
-			(at 130.556 121.666 0)
-			(effects
-				(font
-					(size 1.27 1.27)
-				)
-				(justify left)
+			(at 125.73 121.666 0)
+			(effects
+				(font
+					(size 1.27 1.27)
+				)
+				(justify right)
 			)
 		)
@@
 			(project "BatteryBoard"
 				(path "/b6fd875d-6e05-4440-9a05-0f0aa046a0ef/2701f768-968e-41c8-b7b5-2417f566d99b"
-					(reference "R46")
+					(reference "R39")
 					(unit 1)
 				)
@@
 		(on_board yes)
 		(dnp no)
-		(property "Reference" "Q11"
+		(property "Reference" "Q7"
 			(at 135.89 39.37 90)
 			(effects
@@
 			(project "BatteryBoard"
 				(path "/b6fd875d-6e05-4440-9a05-0f0aa046a0ef/2701f768-968e-41c8-b7b5-2417f566d99b"
-					(reference "Q11")
+					(reference "Q7")
 					(unit 1)
 				)
@@
 		(on_board yes)
 		(dnp no)
-		(property "Reference" "R45"
-			(at 142.24 54.864 0)
-			(effects
-				(font
-					(size 1.27 1.27)
-				)
-				(justify left)
+		(property "Reference" "R38"
+			(at 146.05 54.864 0)
+			(effects
+				(font
+					(size 1.27 1.27)
+				)
+				(justify right)
 			)
 		)
 		(property "Value" "100k"
-			(at 140.97 56.896 0)
-			(effects
-				(font
-					(size 1.27 1.27)
-				)
-				(justify left)
+			(at 146.05 56.896 0)
+			(effects
+				(font
+					(size 1.27 1.27)
+				)
+				(justify right)
 			)
 		)
@@
 			(project "BatteryBoard"
 				(path "/b6fd875d-6e05-4440-9a05-0f0aa046a0ef/2701f768-968e-41c8-b7b5-2417f566d99b"
-					(reference "R45")
+					(reference "R38")
 					(unit 1)
 				)
@@
 		(on_board yes)
 		(dnp no)
-		(property "Reference" "Q14"
+		(property "Reference" "Q10"
 			(at 170.18 104.14 90)
 			(effects
@@
 			(project "BatteryBoard"
 				(path "/b6fd875d-6e05-4440-9a05-0f0aa046a0ef/2701f768-968e-41c8-b7b5-2417f566d99b"
-					(reference "Q14")
-					(unit 1)
-				)
-			)
-		)
-	)
-	(symbol
-		(lib_id "Device:Fuse")
-		(at 113.03 110.49 270)
+					(reference "Q10")
+					(unit 1)
+				)
+			)
+		)
+	)
+	(symbol
+		(lib_id "Device:Fuse_Small")
+		(at 113.03 110.49 180)
 		(unit 1)
 		(exclude_from_sim no)
@@
 		(dnp no)
 		(property "Reference" "F8"
-			(at 113.03 106.172 90)
+			(at 113.03 106.934 0)
 			(effects
 				(font
@@
 		)
 		(property "Value" "6A"
-			(at 113.03 108.204 90)
+			(at 113.03 108.712 0)
 			(effects
 				(font
@@
 		)
 		(property "Footprint" "Fuse:Fuse_1206_3216Metric"
-			(at 113.03 108.712 90)
+			(at 113.03 110.49 0)
 			(effects
 				(font
@@
 			)
 		)
-		(property "Description" "Fuse"
+		(property "Description" "Fuse, small symbol"
 			(at 113.03 110.49 0)
 			(effects
@@
 		)
 		(property "Flight" "0R"
-			(at 113.03 112.776 90)
+			(at 113.03 112.522 0)
 			(effects
 				(font
@@
 		(on_board yes)
 		(dnp no)
-		(property "Reference" "C8"
+		(property "Reference" "C6"
 			(at 150.368 137.414 0)
 			(effects
@@
 			)
 		)
-		(property "Value" "0.1uF"
+		(property "Value" "100n"
 			(at 150.368 139.446 0)
 			(effects
@@
 			(project "BatteryBoard"
 				(path "/b6fd875d-6e05-4440-9a05-0f0aa046a0ef/2701f768-968e-41c8-b7b5-2417f566d99b"
-					(reference "C8")
-					(unit 1)
-				)
-			)
-		)
-	)
-	(symbol
-		(lib_id "Device:Fuse")
-		(at 113.03 45.72 90)
+					(reference "C6")
+					(unit 1)
+				)
+			)
+		)
+	)
+	(symbol
+		(lib_id "Device:Fuse_Small")
+		(at 113.03 45.72 0)
 		(unit 1)
 		(exclude_from_sim no)
@@
 		(dnp no)
 		(property "Reference" "F7"
-			(at 113.03 41.402 90)
+			(at 113.03 42.164 0)
 			(effects
 				(font
@@
 		)
 		(property "Value" "6A"
-			(at 113.03 43.434 90)
+			(at 113.03 43.942 0)
 			(effects
 				(font
@@
 		)
 		(property "Footprint" "Fuse:Fuse_1206_3216Metric"
-			(at 113.03 47.498 90)
+			(at 113.03 45.72 0)
 			(effects
 				(font
@@
 			)
 		)
-		(property "Description" "Fuse"
+		(property "Description" "Fuse, small symbol"
 			(at 113.03 45.72 0)
 			(effects
@@
 		)
 		(property "Flight" "0R"
-			(at 113.03 47.752 90)
+			(at 113.03 47.498 0)
 			(effects
 				(font
@@
 		(on_board yes)
 		(dnp no)
-		(property "Reference" "R47"
+		(property "Reference" "R40"
 			(at 193.04 128.524 0)
 			(effects
@@
 		)
 		(property "Value" "470k"
-			(at 197.866 130.556 0)
-			(effects
-				(font
-					(size 1.27 1.27)
-				)
-				(justify left)
+			(at 193.04 130.556 0)
+			(effects
+				(font
+					(size 1.27 1.27)
+				)
+				(justify right)
 			)
 		)
@@
 			(project "BatteryBoard"
 				(path "/b6fd875d-6e05-4440-9a05-0f0aa046a0ef/2701f768-968e-41c8-b7b5-2417f566d99b"
-					(reference "R47")
+					(reference "R40")
 					(unit 1)
 				)
@@
 		(on_board yes)
 		(dnp no)
-		(property "Reference" "R44"
+		(property "Reference" "R37"
 			(at 118.11 63.754 0)
 			(effects
@@
 			(project "BatteryBoard"
 				(path "/b6fd875d-6e05-4440-9a05-0f0aa046a0ef/2701f768-968e-41c8-b7b5-2417f566d99b"
-					(reference "R44")
+					(reference "R37")
 					(unit 1)
 				)
@@
 		(on_board yes)
 		(dnp no)
-		(property "Reference" "C7"
+		(property "Reference" "C5"
 			(at 188.722 72.644 0)
 			(effects
@@
 			)
 		)
-		(property "Value" "0.1uF"
+		(property "Value" "100n"
 			(at 188.722 74.676 0)
 			(effects
@@
 			(project "BatteryBoard"
 				(path "/b6fd875d-6e05-4440-9a05-0f0aa046a0ef/2701f768-968e-41c8-b7b5-2417f566d99b"
-					(reference "C7")
+					(reference "C5")
 					(unit 1)
 				)
@@
 		(on_board yes)
 		(dnp no)
-		(property "Reference" "U4"
+		(property "Reference" "U3"
 			(at 170.942 55.88 0)
 			(effects
@@
 			(project ""
 				(path "/b6fd875d-6e05-4440-9a05-0f0aa046a0ef/2701f768-968e-41c8-b7b5-2417f566d99b"
-					(reference "U4")
+					(reference "U3")
 					(unit 1)
 				)
@@
 		(on_board yes)
 		(dnp no)
-		(property "Reference" "Q13"
+		(property "Reference" "Q9"
 			(at 135.89 104.14 90)
 			(effects
@@
 			(project "BatteryBoard"
 				(path "/b6fd875d-6e05-4440-9a05-0f0aa046a0ef/2701f768-968e-41c8-b7b5-2417f566d99b"
-					(reference "Q13")
+					(reference "Q9")
 					(unit 1)
 				)
@@
 		(dnp no)
 		(fields_autoplaced yes)
-		(property "Reference" "U5"
-			(at 172.3741 120.65 0)
+		(property "Reference" "U4"
+			(at 172.3233 120.65 0)
 			(effects
 				(font
@@
 		)
 		(property "Value" "LTC4412xS6"
-			(at 172.3741 123.19 0)
+			(at 172.3233 123.19 0)
 			(effects
 				(font
@@
 			(project ""
 				(path "/b6fd875d-6e05-4440-9a05-0f0aa046a0ef/2701f768-968e-41c8-b7b5-2417f566d99b"
-					(reference "U5")
+					(reference "U4")
 					(unit 1)
 				)
@@
 		(on_board yes)
 		(dnp no)
-		(property "Reference" "Q12"
+		(property "Reference" "Q8"
 			(at 168.91 39.37 90)
 			(effects
@@
 			(project ""
 				(path "/b6fd875d-6e05-4440-9a05-0f0aa046a0ef/2701f768-968e-41c8-b7b5-2417f566d99b"
-					(reference "Q12")
-					(unit 1)
-				)
+					(reference "Q8")
+					(unit 1)
+				)

Commit message: Idk some changes
Parts:
- C5, C6: MPN (none) -> C307348
- F7, F8: MPN (none) -> C844862
- Q10, Q7, Q8, Q9: MPN (none) -> C3289459
- R37, R40: MPN (none) -> C138280
- R38, R39: MPN (none) -> C237792
Changed lines of the file:
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@@
+			)
+		)
+		(property "MPN" "C237792"
+			(at 124.46 120.65 0)
+			(effects
+				(font
+					(size 1.27 1.27)
+				)
+				(hide yes)
 			)
 		)
@@
 			)
 		)
+		(property "MPN" "C3289459"
+			(at 135.89 48.26 90)
+			(effects
+				(font
+					(size 1.27 1.27)
+				)
+				(hide yes)
+			)
+		)
 		(pin "5"
 		)
@@
 			)
 		)
+		(property "MPN" "C237792"
+			(at 147.32 55.88 0)
+			(effects
+				(font
+					(size 1.27 1.27)
+				)
+				(hide yes)
+			)
+		)
 		(pin "2"
 		)
@@
 			)
 		)
+		(property "MPN" "C3289459"
+			(at 170.18 113.03 90)
+			(effects
+				(font
+					(size 1.27 1.27)
+				)
+				(hide yes)
+			)
+		)
 		(pin "5"
 		)
@@
 					(size 1.27 1.27)
 				)
+			)
+		)
+		(property "MPN" "C844862"
+			(at 113.03 110.49 0)
+			(effects
+				(font
+					(size 1.27 1.27)
+				)
+				(hide yes)
 			)
 		)
@@
 			)
 		)
+		(property "MPN" "C307348"
+			(at 152.4 138.43 0)
+			(effects
+				(font
+					(size 1.27 1.27)
+				)
+				(hide yes)
+			)
+		)
 		(pin "2"
 		)
@@
 					(size 1.27 1.27)
 				)
+			)
+		)
+		(property "MPN" "C844862"
+			(at 113.03 45.72 0)
+			(effects
+				(font
+					(size 1.27 1.27)
+				)
+				(hide yes)
 			)
 		)
@@
 			)
 		)
+		(property "MPN" "C138280"
+			(at 191.77 129.54 0)
+			(effects
+				(font
+					(size 1.27 1.27)
+				)
+				(hide yes)
+			)
+		)
 		(pin "2"
 		)
@@
 			)
 		)
+		(property "MPN" "C138280"
+			(at 119.38 64.77 0)
+			(effects
+				(font
+					(size 1.27 1.27)
+				)
+				(hide yes)
+			)
+		)
 		(pin "2"
 		)
@@
 		)
 		(property "Description" "Unpolarized capacitor, small symbol"
+			(at 186.69 73.66 0)
+			(effects
+				(font
+					(size 1.27 1.27)
+				)
+				(hide yes)
+			)
+		)
+		(property "MPN" "C307348"
 			(at 186.69 73.66 0)
 			(effects
@@
 			)
 		)
+		(property "MPN" "C3289459"
+			(at 135.89 113.03 90)
+			(effects
+				(font
+					(size 1.27 1.27)
+				)
+				(hide yes)
+			)
+		)
 		(pin "5"
 		)
@@
 			(effects
 				(font
+					(size 1.27 1.27)
+				)
+				(hide yes)
+			)
+		)
+		(property "MPN" "C3289459"
+			(at 168.91 48.26 90)
+			(effects
+				(font
