File: BatteryBusProtection.kicad_sch (KiCad schematic)
At the start: 16 parts, among them Q10 SIRA99DP-T1-GE3, Q7 SIRA99DP-T1-GE3, Q8 SIRA99DP-T1-GE3, Q9 SIRA99DP-T1-GE3, U3 LTC4412xS6, U4 LTC4412xS6

Commit message: making a few changes
Other:
- title: Argus Batteryboard -> Batteryboard
Changed lines of the file:
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@@
 	(paper "USLetter")
 	(title_block
-		(title "Argus Batteryboard")
-		(date "2026-04-14")
-		(rev "v3.2")
+		(title "Batteryboard")
+		(date "2026-08-21")
+		(rev "v4.0")
 		(company "Carnegie Mellon University")
-		(comment 1 "M. Holliday")
-		(comment 2 "N. Khera")
-		(comment 3 "V. Rajesh")
+		(comment 1 "N. Khera")
+		(comment 2 "V. Rajesh")
+		(comment 3 "S. Farhan")
 	)
 	(rectangle

Commit message: routing
Parts:
- renumbered C5 to C10, C6 to C11, F7 to F5, F8 to F6, Q7 to Q1, Q8 to Q2, Q9 to Q3, Q10 to Q4, R66 to R20, R38 to R21, R37 to R22, R67 to R23, R39 to R24, R40 to R25, U3 to U4, U4 to U5
Changed lines of the file:
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@@
 		(in_pos_files yes)
 		(dnp no)
-		(property "Reference" "R39"
+		(property "Reference" "R24"
 			(at 125.73 119.634 0)
 			(show_name no)
@@
 			(project "Avionics-BatteryBoard"
 				(path "/b6fd875d-6e05-4440-9a05-0f0aa046a0ef/2701f768-968e-41c8-b7b5-2417f566d99b"
-					(reference "R39")
+					(reference "R24")
 					(unit 1)
 				)
@@
 		(in_pos_files yes)
 		(dnp no)
-		(property "Reference" "R66"
+		(property "Reference" "R20"
 			(at 135.89 33.02 90)
 			(show_name no)
@@
 			(project "Avionics-BatteryBoard"
 				(path "/b6fd875d-6e05-4440-9a05-0f0aa046a0ef/2701f768-968e-41c8-b7b5-2417f566d99b"
-					(reference "R66")
+					(reference "R20")
 					(unit 1)
 				)
@@
 		(in_pos_files yes)
 		(dnp no)
-		(property "Reference" "#PWR019"
+		(property "Reference" "#PWR010"
 			(at 119.38 63.5 0)
 			(hide yes)
@@
 			(project "Avionics-BatteryBoard"
 				(path "/b6fd875d-6e05-4440-9a05-0f0aa046a0ef/2701f768-968e-41c8-b7b5-2417f566d99b"
-					(reference "#PWR019")
+					(reference "#PWR010")
 					(unit 1)
 				)
@@
 		(in_pos_files yes)
 		(dnp yes)
-		(property "Reference" "Q7"
+		(property "Reference" "Q1"
 			(at 135.89 40.64 90)
 			(show_name no)
@@
 			(project "Avionics-BatteryBoard"
 				(path "/b6fd875d-6e05-4440-9a05-0f0aa046a0ef/2701f768-968e-41c8-b7b5-2417f566d99b"
-					(reference "Q7")
+					(reference "Q1")
 					(unit 1)
 				)
@@
 		(in_pos_files yes)
 		(dnp no)
-		(property "Reference" "R38"
+		(property "Reference" "R21"
 			(at 146.05 54.864 0)
 			(show_name no)
@@
 			(project "Avionics-BatteryBoard"
 				(path "/b6fd875d-6e05-4440-9a05-0f0aa046a0ef/2701f768-968e-41c8-b7b5-2417f566d99b"
-					(reference "R38")
+					(reference "R21")
 					(unit 1)
 				)
@@
 		(in_pos_files yes)
 		(dnp no)
-		(property "Reference" "Q10"
+		(property "Reference" "Q4"
 			(at 170.18 105.41 90)
 			(show_name no)
@@
 			(project "Avionics-BatteryBoard"
 				(path "/b6fd875d-6e05-4440-9a05-0f0aa046a0ef/2701f768-968e-41c8-b7b5-2417f566d99b"
-					(reference "Q10")
+					(reference "Q4")
 					(unit 1)
 				)
@@
 		(in_pos_files yes)
 		(dnp no)
-		(property "Reference" "F8"
+		(property "Reference" "F6"
 			(at 113.03 106.934 0)
 			(show_name no)
@@
 			(project "Avionics-BatteryBoard"
 				(path "/b6fd875d-6e05-4440-9a05-0f0aa046a0ef/2701f768-968e-41c8-b7b5-2417f566d99b"
-					(reference "F8")
+					(reference "F6")
 					(unit 1)
 				)
@@
 		(in_pos_files yes)
 		(dnp no)
-		(property "Reference" "C6"
+		(property "Reference" "C11"
 			(at 150.368 137.414 0)
 			(show_name no)
@@
 			(project "Avionics-BatteryBoard"
 				(path "/b6fd875d-6e05-4440-9a05-0f0aa046a0ef/2701f768-968e-41c8-b7b5-2417f566d99b"
-					(reference "C6")
+					(reference "C11")
 					(unit 1)
 				)
@@
 		(in_pos_files yes)
 		(dnp no)
-		(property "Reference" "F7"
+		(property "Reference" "F5"
 			(at 113.03 42.164 0)
 			(show_name no)
@@
 			(project "Avionics-BatteryBoard"
 				(path "/b6fd875d-6e05-4440-9a05-0f0aa046a0ef/2701f768-968e-41c8-b7b5-2417f566d99b"
-					(reference "F7")
+					(reference "F5")
 					(unit 1)
 				)
@@
 		(in_pos_files yes)
 		(dnp no)
-		(property "Reference" "R40"
+		(property "Reference" "R25"
 			(at 193.04 128.524 0)
 			(show_name no)
@@
 			(project "Avionics-BatteryBoard"
 				(path "/b6fd875d-6e05-4440-9a05-0f0aa046a0ef/2701f768-968e-41c8-b7b5-2417f566d99b"
-					(reference "R40")
+					(reference "R25")
 					(unit 1)
 				)
@@
 		(in_pos_files yes)
 		(dnp no)
-		(property "Reference" "R37"
+		(property "Reference" "R22"
 			(at 118.11 63.754 0)
 			(show_name no)
@@
 			(project "Avionics-BatteryBoard"
 				(path "/b6fd875d-6e05-4440-9a05-0f0aa046a0ef/2701f768-968e-41c8-b7b5-2417f566d99b"
-					(reference "R37")
+					(reference "R22")
 					(unit 1)
 				)
@@
 		(in_pos_files yes)
 		(dnp yes)
-		(property "Reference" "R67"
+		(property "Reference" "R23"
 			(at 135.89 97.79 90)
 			(show_name no)
@@
 			(project "Avionics-BatteryBoard"
 				(path "/b6fd875d-6e05-4440-9a05-0f0aa046a0ef/2701f768-968e-41c8-b7b5-2417f566d99b"
-					(reference "R67")
+					(reference "R23")
 					(unit 1)
 				)
@@
 		(in_pos_files yes)
 		(dnp no)
-		(property "Reference" "C5"
+		(property "Reference" "C10"
 			(at 189.992 72.644 0)
 			(show_name no)
@@
 			(project "Avionics-BatteryBoard"
 				(path "/b6fd875d-6e05-4440-9a05-0f0aa046a0ef/2701f768-968e-41c8-b7b5-2417f566d99b"
-					(reference "C5")
+					(reference "C10")
 					(unit 1)
 				)
@@
 		(in_pos_files yes)
 		(dnp no)
-		(property "Reference" "#PWR050"
+		(property "Reference" "#PWR09"
 			(at 204.47 46.99 0)
 			(hide yes)
@@
 			(project "Avionics-BatteryBoard"
 				(path "/b6fd875d-6e05-4440-9a05-0f0aa046a0ef/2701f768-968e-41c8-b7b5-2417f566d99b"
-					(reference "#PWR050")
+					(reference "#PWR09")
 					(unit 1)
 				)
@@
 		(in_pos_files yes)
 		(dnp no)
-		(property "Reference" "U3"
+		(property "Reference" "U4"
 			(at 172.212 55.88 0)
 			(show_name no)
@@
 			(project "Avionics-BatteryBoard"
 				(path "/b6fd875d-6e05-4440-9a05-0f0aa046a0ef/2701f768-968e-41c8-b7b5-2417f566d99b"
-					(reference "U3")
+					(reference "U4")
 					(unit 1)
 				)
@@
 		(in_pos_files yes)
 		(dnp no)
-		(property "Reference" "#PWR03"
+		(property "Reference" "#PWR013"
 			(at 170.18 154.94 0)
 			(hide yes)
@@
 			(project "Avionics-BatteryBoard"
 				(path "/b6fd875d-6e05-4440-9a05-0f0aa046a0ef/2701f768-968e-41c8-b7b5-2417f566d99b"
-					(reference "#PWR03")
+					(reference "#PWR013")
 					(unit 1)
 				)
@@
 		(in_pos_files yes)
 		(dnp no)
-		(property "Reference" "Q9"
+		(property "Reference" "Q3"
 			(at 135.89 105.41 90)
 			(show_name no)
@@
 			(project "Avionics-BatteryBoard"
 				(path "/b6fd875d-6e05-4440-9a05-0f0aa046a0ef/2701f768-968e-41c8-b7b5-2417f566d99b"
-					(reference "Q9")
+					(reference "Q3")
 					(unit 1)
 				)
@@
 		(dnp no)
 		(fields_autoplaced yes)
-		(property "Reference" "U4"
+		(property "Reference" "U5"
 			(at 172.3233 120.65 0)
 			(show_name no)
@@
 			(project "Avionics-BatteryBoard"
 				(path "/b6fd875d-6e05-4440-9a05-0f0aa046a0ef/2701f768-968e-41c8-b7b5-2417f566d99b"
-					(reference "U4")
+					(reference "U5")
 					(unit 1)
 				)
@@
 		(in_pos_files yes)
 		(dnp no)
-		(property "Reference" "Q8"
+		(property "Reference" "Q2"
 			(at 170.18 40.64 90)
 			(show_name no)
@@
 			(project "Avionics-BatteryBoard"
 				(path "/b6fd875d-6e05-4440-9a05-0f0aa046a0ef/2701f768-968e-41c8-b7b5-2417f566d99b"
-					(reference "Q8")
+					(reference "Q2")
 					(unit 1)
 				)
@@
 		(in_pos_files yes)
 		(dnp no)
-		(property "Reference" "#PWR01"
+		(property "Reference" "#PWR011"
 			(at 170.18 90.17 0)
 			(hide yes)
@@
 			(project "Avionics-BatteryBoard"
 				(path "/b6fd875d-6e05-4440-9a05-0f0aa046a0ef/2701f768-968e-41c8-b7b5-2417f566d99b"
-					(reference "#PWR01")
-					(unit 1)
-				)
+					(reference "#PWR011")
+					(unit 1)
+				)
