File: BatteryMonitor.kicad_sch (KiCad schematic)
At the start: 26 parts, among them J5 Fuel Gauge Programming Header, U6 MAX17205

Commit message: v3.1 Updates
Parts:
- C10: renamed from C12; value 0.47uF -> 470n
- C11: renamed from C13; value 0.47uF -> 470n
- C7: renamed from C9; value 1nF -> 1n
- C8: renamed from C10; value 1nF -> 1n
- C9: renamed from C11; value 0.1uF -> 100n
- R47: renamed from R54; value 51.1k -> 51k1
- renumbered R48 to R41, R49 to R42, R50 to R43, R51 to R44, R52 to R45, R53 to R46, R55 to R48, R56 to R49, R57 to R50, R58 to R51, R59 to R52, R60 to R53, U6 to U5
Other:
- note added: "Rsense"
- note removed: "Remove before programming"
Changed lines of the file:
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@@
 		)
 	)
-	(text "Remove before programming"
+	(text "Rsense"
 		(exclude_from_sim no)
-		(at 195.072 131.064 0)
+		(at 101.6 70.866 0)
 		(effects
 			(font
@@
 	)
 	(junction
-		(at 78.74 99.06)
+		(at 110.49 68.58)
 		(diameter 0)
 		(color 0 0 0 0)
 	)
 	(junction
-		(at 67.31 88.9)
+		(at 78.74 99.06)
 		(diameter 0)
 		(color 0 0 0 0)
 	)
 	(junction
-		(at 144.78 111.76)
+		(at 67.31 88.9)
 		(diameter 0)
 		(color 0 0 0 0)
 	)
 	(junction
-		(at 109.22 68.58)
+		(at 144.78 111.76)
 		(diameter 0)
 		(color 0 0 0 0)
@@
 	(wire
 		(pts
-			(xy 109.22 68.58) (xy 144.78 68.58)
-		)
-		(stroke
-			(width 0)
-			(type default)
-		)
-	)
-	(wire
-		(pts
 			(xy 198.12 82.55) (xy 185.42 82.55)
 		)
@@
 	(wire
 		(pts
-			(xy 106.68 73.66) (xy 109.22 73.66)
+			(xy 106.68 73.66) (xy 110.49 73.66)
 		)
 		(stroke
@@
 	(wire
 		(pts
-			(xy 109.22 73.66) (xy 109.22 68.58)
+			(xy 110.49 73.66) (xy 110.49 68.58)
 		)
 		(stroke
@@
 	(wire
 		(pts
+			(xy 110.49 68.58) (xy 144.78 68.58)
+		)
+		(stroke
+			(width 0)
+			(type default)
+		)
+	)
+	(wire
+		(pts
 			(xy 144.78 104.14) (xy 144.78 111.76)
 		)
@@
 	(wire
 		(pts
-			(xy 104.14 68.58) (xy 109.22 68.58)
+			(xy 104.14 68.58) (xy 110.49 68.58)
 		)
 		(stroke
@@
 		(on_board yes)
 		(dnp no)
-		(property "Reference" "R56"
+		(property "Reference" "R49"
 			(at 196.088 78.74 90)
 			(effects
@@
 			(project "BatteryBoard"
 				(path "/b6fd875d-6e05-4440-9a05-0f0aa046a0ef/ad142cc2-d77f-4a6c-99c2-d9e17f4c27ae"
-					(reference "R56")
+					(reference "R49")
 					(unit 1)
 				)
@@
 		(on_board yes)
 		(dnp no)
-		(property "Reference" "R60"
-			(at 194.31 125.984 90)
+		(property "Reference" "R53"
+			(at 194.564 124.206 90)
 			(effects
 				(font
@@
 		)
 		(property "Value" "0R"
-			(at 194.31 123.952 90)
+			(at 194.564 126.238 90)
 			(effects
 				(font
@@
 			(project "BatteryBoard"
 				(path "/b6fd875d-6e05-4440-9a05-0f0aa046a0ef/ad142cc2-d77f-4a6c-99c2-d9e17f4c27ae"
-					(reference "R60")
+					(reference "R53")
 					(unit 1)
 				)
@@
 		(on_board yes)
 		(dnp no)
-		(property "Reference" "R50"
+		(property "Reference" "R43"
 			(at 101.6 64.262 90)
 			(effects
@@
 			(project ""
 				(path "/b6fd875d-6e05-4440-9a05-0f0aa046a0ef/ad142cc2-d77f-4a6c-99c2-d9e17f4c27ae"
-					(reference "R50")
+					(reference "R43")
 					(unit 1)
 				)
@@
 		(on_board yes)
 		(dnp no)
-		(property "Reference" "R55"
+		(property "Reference" "R48"
 			(at 196.088 73.66 90)
 			(effects
@@
 			(project "BatteryBoard"
 				(path "/b6fd875d-6e05-4440-9a05-0f0aa046a0ef/ad142cc2-d77f-4a6c-99c2-d9e17f4c27ae"
-					(reference "R55")
+					(reference "R48")
 					(unit 1)
 				)
@@
 		(on_board yes)
 		(dnp no)
-		(property "Reference" "R53"
-			(at 146.304 100.584 0)
+		(property "Reference" "R46"
+			(at 146.05 100.584 0)
 			(effects
 				(font
@@
 		)
 		(property "Value" "30k"
-			(at 146.304 102.616 0)
+			(at 146.05 102.616 0)
 			(effects
 				(font
@@
 			(project "BatteryBoard"
 				(path "/b6fd875d-6e05-4440-9a05-0f0aa046a0ef/ad142cc2-d77f-4a6c-99c2-d9e17f4c27ae"
-					(reference "R53")
+					(reference "R46")
 					(unit 1)
 				)
@@
 		(on_board yes)
 		(dnp no)
-		(property "Reference" "R58"
+		(property "Reference" "R51"
 			(at 194.31 102.616 90)
 			(effects
@@
 			(project "BatteryBoard"
 				(path "/b6fd875d-6e05-4440-9a05-0f0aa046a0ef/ad142cc2-d77f-4a6c-99c2-d9e17f4c27ae"
-					(reference "R58")
+					(reference "R51")
 					(unit 1)
 				)
@@
 		(on_board yes)
 		(dnp no)
-		(property "Reference" "R48"
+		(property "Reference" "R41"
 			(at 46.99 84.836 90)
 			(effects
@@
 			(project ""
 				(path "/b6fd875d-6e05-4440-9a05-0f0aa046a0ef/ad142cc2-d77f-4a6c-99c2-d9e17f4c27ae"
-					(reference "R48")
+					(reference "R41")
 					(unit 1)
 				)
@@
 		(on_board yes)
 		(dnp no)
-		(property "Reference" "C9"
-			(at 59.436 92.964 0)
+		(property "Reference" "C7"
+			(at 59.182 92.964 0)
 			(effects
 				(font
@@
 			)
 		)
-		(property "Value" "1nF"
-			(at 59.436 94.996 0)
+		(property "Value" "1n"
+			(at 59.182 94.996 0)
 			(effects
 				(font
@@
 			(project ""
 				(path "/b6fd875d-6e05-4440-9a05-0f0aa046a0ef/ad142cc2-d77f-4a6c-99c2-d9e17f4c27ae"
-					(reference "C9")
+					(reference "C7")
 					(unit 1)
 				)
@@
 		(on_board yes)
 		(dnp no)
-		(property "Reference" "C12"
-			(at 99.314 120.904 0)
+		(property "Reference" "C10"
+			(at 99.568 120.904 0)
 			(effects
 				(font
@@
 			)
 		)
-		(property "Value" "0.47uF"
-			(at 99.314 122.936 0)
+		(property "Value" "470n"
+			(at 99.568 122.936 0)
 			(effects
 				(font
@@
 			(project "BatteryBoard"
 				(path "/b6fd875d-6e05-4440-9a05-0f0aa046a0ef/ad142cc2-d77f-4a6c-99c2-d9e17f4c27ae"
-					(reference "C12")
+					(reference "C10")
 					(unit 1)
 				)
@@
 		(on_board yes)
 		(dnp no)
-		(property "Reference" "R51"
+		(property "Reference" "R44"
 			(at 125.73 87.63 90)
 			(effects
@@
 			(project "BatteryBoard"
 				(path "/b6fd875d-6e05-4440-9a05-0f0aa046a0ef/ad142cc2-d77f-4a6c-99c2-d9e17f4c27ae"
-					(reference "R51")
+					(reference "R44")
 					(unit 1)
 				)
@@
 		(on_board yes)
 		(dnp no)
-		(property "Reference" "R57"
+		(property "Reference" "R50"
 			(at 196.088 81.534 90)
 			(effects
@@
 			(project "BatteryBoard"
 				(path "/b6fd875d-6e05-4440-9a05-0f0aa046a0ef/ad142cc2-d77f-4a6c-99c2-d9e17f4c27ae"
-					(reference "R57")
+					(reference "R50")
 					(unit 1)
 				)
@@
 		(on_board yes)
 		(dnp no)
-		(property "Reference" "C13"
-			(at 108.966 120.904 0)
+		(property "Reference" "C11"
+			(at 108.712 120.904 0)
 			(effects
 				(font
@@
 			)
 		)
-		(property "Value" "0.47uF"
-			(at 108.966 122.936 0)
+		(property "Value" "470n"
+			(at 108.712 122.936 0)
 			(effects
 				(font
@@
 			(project "BatteryBoard"
 				(path "/b6fd875d-6e05-4440-9a05-0f0aa046a0ef/ad142cc2-d77f-4a6c-99c2-d9e17f4c27ae"
-					(reference "C13")
+					(reference "C11")
 					(unit 1)
 				)
@@
 		(on_board yes)
 		(dnp no)
-		(property "Reference" "R54"
+		(property "Reference" "R47"
 			(at 196.088 71.12 90)
 			(effects
@@
 			)
 		)
-		(property "Value" "51.1k"
+		(property "Value" "51k1"
 			(at 205.486 71.12 90)
 			(effects
@@
 			(project "BatteryBoard"
 				(path "/b6fd875d-6e05-4440-9a05-0f0aa046a0ef/ad142cc2-d77f-4a6c-99c2-d9e17f4c27ae"
-					(reference "R54")
+					(reference "R47")
 					(unit 1)
 				)
@@
 		(on_board yes)
 		(dnp no)
-		(property "Reference" "R59"
+		(property "Reference" "R52"
 			(at 194.31 112.776 90)
 			(effects
@@
 			(project "BatteryBoard"
 				(path "/b6fd875d-6e05-4440-9a05-0f0aa046a0ef/ad142cc2-d77f-4a6c-99c2-d9e17f4c27ae"
-					(reference "R59")
+					(reference "R52")
 					(unit 1)
 				)
@@
 		(on_board yes)
 		(dnp no)
-		(property "Reference" "R49"
+		(property "Reference" "R42"
 			(at 46.99 94.996 90)
 			(effects
@@
 			(project ""
 				(path "/b6fd875d-6e05-4440-9a05-0f0aa046a0ef/ad142cc2-d77f-4a6c-99c2-d9e17f4c27ae"
-					(reference "R49")
+					(reference "R42")
 					(unit 1)
 				)
@@
 		(on_board yes)
 		(dnp no)
-		(property "Reference" "C10"
-			(at 59.436 103.124 0)
+		(property "Reference" "C8"
+			(at 59.182 103.124 0)
 			(effects
 				(font
@@
 			)
 		)
-		(property "Value" "1nF"
-			(at 59.436 105.156 0)
+		(property "Value" "1n"
+			(at 59.182 105.156 0)
 			(effects
 				(font
@@
 			(project ""
 				(path "/b6fd875d-6e05-4440-9a05-0f0aa046a0ef/ad142cc2-d77f-4a6c-99c2-d9e17f4c27ae"
-					(reference "C10")
+					(reference "C8")
 					(unit 1)
 				)
@@
 		(on_board yes)
 		(dnp no)
-		(property "Reference" "U6"
+		(property "Reference" "U5"
 			(at 101.6 95.504 0)
 			(effects
@@
 			(project "BatteryBoard"
 				(path "/b6fd875d-6e05-4440-9a05-0f0aa046a0ef/ad142cc2-d77f-4a6c-99c2-d9e17f4c27ae"
-					(reference "U6")
+					(reference "U5")
 					(unit 1)
 				)
@@
 		(on_board yes)
 		(dnp no)
-		(property "Reference" "R52"
+		(property "Reference" "R45"
 			(at 133.35 100.584 0)
 			(effects
@@
 			(project ""
 				(path "/b6fd875d-6e05-4440-9a05-0f0aa046a0ef/ad142cc2-d77f-4a6c-99c2-d9e17f4c27ae"
-					(reference "R52")
+					(reference "R45")
 					(unit 1)
 				)
@@
 		(on_board yes)
 		(dnp no)
-		(property "Reference" "C11"
-			(at 69.596 92.964 0)
+		(property "Reference" "C9"
+			(at 69.342 92.964 0)
 			(effects
 				(font
@@
 			)
 		)
-		(property "Value" "0.1uF"
-			(at 69.596 94.996 0)
+		(property "Value" "100n"
+			(at 69.342 94.996 0)
 			(effects
 				(font
@@
 			(project "BatteryBoard"
 				(path "/b6fd875d-6e05-4440-9a05-0f0aa046a0ef/ad142cc2-d77f-4a6c-99c2-d9e17f4c27ae"
-					(reference "C11")
+					(reference "C9")
 					(unit 1)
 				)

Commit message: Idk some changes
Parts:
- C10, C11: MPN (none) -> C472773
- C7, C8: MPN (none) -> C161231
- C9: MPN (none) -> C307348
- R41: MPN (none) -> C3029194
- R42: MPN (none) -> C844917
- R43: MPN (none) -> C840621
- R44: MPN (none) -> C2484712
- R45, R46: MPN (none) -> C844774
- R47: MPN (none) -> C844575
- R48, R49, R50: MPN (none) -> C844741
- R51: MPN (none) -> C2479067
- R52, R53: MPN (none) -> C844915
- TH1: Field5 (none) -> NTCS0603E3103JLT
- U5: MPN (none) -> C401140
Changed lines of the file:
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@@
+			)
+		)
+		(property "MPN" "C844741"
+			(at 200.66 80.01 90)
+			(effects
+				(font
+					(size 1.27 1.27)
+				)
+				(hide yes)
 			)
 		)
@@
 			)
 		)
+		(property "MPN" "C844915"
+			(at 194.31 121.92 90)
+			(effects
+				(font
+					(size 1.27 1.27)
+				)
+				(hide yes)
+			)
+		)
 		(pin "1"
 		)
@@
 		(property "Description" "Resistor, small symbol"
 			(at 101.6 68.58 0)
+			(effects
+				(font
+					(size 1.27 1.27)
+				)
+				(hide yes)
+			)
+		)
+		(property "MPN" "C840621"
+			(at 101.6 68.58 90)
 			(effects
 				(font
@@
 			)
 		)
+		(property "MPN" "C844741"
+			(at 200.66 74.93 90)
+			(effects
+				(font
+					(size 1.27 1.27)
+				)
+				(hide yes)
+			)
+		)
 		(pin "1"
 		)
@@
 			)
 		)
+		(property "MPN" "C844774"
+			(at 144.78 101.6 0)
+			(effects
+				(font
+					(size 1.27 1.27)
+				)
+				(hide yes)
+			)
+		)
 		(pin "1"
 		)
@@
 		(property "Description" "Resistor, small symbol"
 			(at 194.31 106.68 0)
+			(effects
+				(font
+					(size 1.27 1.27)
+				)
+				(hide yes)
+			)
+		)
+		(property "MPN" "C2479067"
+			(at 194.31 106.68 90)
 			(effects
 				(font
@@
 			)
 		)
+		(property "MPN" "C3029194"
+			(at 46.99 88.9 90)
+			(effects
+				(font
+					(size 1.27 1.27)
+				)
+				(hide yes)
+			)
+		)
 		(pin "1"
 		)
@@
 		)
 		(property "Description" "Unpolarized capacitor, small symbol"
+			(at 57.15 93.98 0)
+			(effects
+				(font
+					(size 1.27 1.27)
+				)
+				(hide yes)
+			)
+		)
+		(property "MPN" "C161231"
 			(at 57.15 93.98 0)
 			(effects
@@
 			)
 		)
+		(property "MPN" "C472773"
+			(at 101.6 121.92 0)
+			(effects
+				(font
+					(size 1.27 1.27)
+				)
+				(hide yes)
+			)
+		)
 		(pin "2"
 		)
@@
 			)
 		)
+		(property "MPN" "C2484712"
+			(at 125.73 91.44 90)
+			(effects
+				(font
+					(size 1.27 1.27)
+				)
+				(hide yes)
+			)
+		)
 		(pin "1"
 		)
@@
 			)
 		)
+		(property "MPN" "C844741"
+			(at 200.66 82.55 90)
+			(effects
+				(font
+					(size 1.27 1.27)
+				)
+				(hide yes)
+			)
+		)
 		(pin "1"
 		)
@@
 		)
 		(property "Description" "Unpolarized capacitor, small symbol"
+			(at 106.68 121.92 0)
+			(effects
+				(font
+					(size 1.27 1.27)
+				)
+				(hide yes)
+			)
+		)
+		(property "MPN" "C472773"
 			(at 106.68 121.92 0)
 			(effects
@@
 			)
 		)
+		(property "Field5" "NTCS0603E3103JLT"
+			(at 138.43 152.146 0)
+			(effects
+				(font
+					(size 1.27 1.27)
+				)
+			)
+		)
 		(pin "2"
 		)
@@
 			)
 		)
+		(property "MPN" "C844575"
+			(at 200.66 72.39 90)
+			(effects
+				(font
+					(size 1.27 1.27)
+				)
+				(hide yes)
+			)
+		)
 		(pin "1"
 		)
@@
 		(property "Description" "Resistor, small symbol"
 			(at 194.31 116.84 0)
+			(effects
+				(font
+					(size 1.27 1.27)
+				)
+				(hide yes)
+			)
+		)
+		(property "MPN" "C844915"
+			(at 194.31 116.84 90)
 			(effects
 				(font
@@
 			)
 		)
+		(property "MPN" "C844917"
+			(at 46.99 99.06 90)
+			(effects
+				(font
+					(size 1.27 1.27)
+				)
+				(hide yes)
+			)
+		)
 		(pin "1"
 		)
@@
 			)
 		)
+		(property "MPN" "C161231"
+			(at 57.15 104.14 0)
+			(effects
+				(font
+					(size 1.27 1.27)
+				)
+				(hide yes)
+			)
+		)
 		(pin "2"
 		)
@@
 			)
 		)
+		(property "MPN" "C401140"
+			(at 101.6 96.52 0)
+			(effects
+				(font
+					(size 1.27 1.27)
+				)
+				(hide yes)
+			)
+		)
 		(pin "5"
 		)
@@
 			)
 		)
+		(property "MPN" "C844774"
+			(at 132.08 101.6 0)
+			(effects
+				(font
+					(size 1.27 1.27)
+				)
+				(hide yes)
+			)
+		)
 		(pin "1"
 		)
@@
 			(at 67.31 93.98 0)
 			(effects
+				(font
+					(size 1.27 1.27)
+				)
+				(hide yes)
+			)
+		)
+		(property "MPN" "C307348"
+			(at 67.31 93.98 0)
+			(effects
