File: BatteryMonitor.kicad_sch (KiCad schematic)
At the start: 26 parts, among them J5 Fuel Gauge Programming Header, U5 MAX17205

Commit message: making a few changes
Parts:
- removed TH3, TH6: 10k 3435k, Capacitor_SMD:C_0603_1608Metric, symbol Device:Thermistor_NTC
Connections:
- net SYSTEM_VSS: now also TH2.2, TH5.2
Other:
- title: Argus Batteryboard -> Batteryboard
Changed lines of the file:
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@@
 	(paper "USLetter")
 	(title_block
-		(title "Argus Batteryboard")
-		(date "2026-04-14")
-		(rev "v3.2")
+		(title "Batteryboard")
+		(date "2026-08-21")
+		(rev "v4.0")
 		(company "Carnegie Mellon University")
-		(comment 1 "M. Holliday")
-		(comment 2 "N. Khera")
-		(comment 3 "V. Rajesh")
+		(comment 1 "N. Khera")
+		(comment 2 "V. Rajesh")
+		(comment 3 "S. Farhan")
 	)
 	(rectangle
@@
 	(wire
 		(pts
-			(xy 132.08 143.51) (xy 132.08 146.05)
-		)
-		(stroke
-			(width 0)
-			(type default)
-		)
-	)
-	(wire
-		(pts
 			(xy 203.2 82.55) (xy 215.9 82.55)
 		)
@@
 	(wire
 		(pts
-			(xy 132.08 133.35) (xy 132.08 135.89)
+			(xy 132.08 133.35) (xy 132.08 138.43)
 		)
 		(stroke
@@
 	(wire
 		(pts
-			(xy 144.78 133.35) (xy 144.78 135.89)
-		)
-		(stroke
-			(width 0)
-			(type default)
-		)
-	)
-	(wire
-		(pts
 			(xy 210.82 77.47) (xy 210.82 86.36)
 		)
@@
 	(wire
 		(pts
-			(xy 144.78 143.51) (xy 144.78 146.05)
+			(xy 144.78 133.35) (xy 144.78 138.43)
 		)
 		(stroke
@@
 	)
 	(symbol
-		(lib_id "Device:Thermistor_NTC")
-		(at 144.78 139.7 0)
-		(unit 1)
-		(body_style 1)
-		(exclude_from_sim no)
-		(in_bom yes)
-		(on_board yes)
-		(in_pos_files yes)
-		(dnp no)
-		(fields_autoplaced yes)
-		(property "Reference" "TH6"
-			(at 147.32 138.7474 0)
-			(show_name no)
-			(do_not_autoplace no)
-			(effects
-				(font
-					(size 1.27 1.27)
-				)
-				(justify left)
-			)
-		)
-		(property "Value" "10k 3435k"
-			(at 147.32 141.2874 0)
-			(show_name no)
-			(do_not_autoplace no)
-			(effects
-				(font
-					(size 1.27 1.27)
-				)
-				(justify left)
-			)
-		)
-		(property "Footprint" "Capacitor_SMD:C_0603_1608Metric"
-			(at 144.78 138.43 0)
-			(hide yes)
-			(show_name no)
-			(do_not_autoplace no)
-			(effects
-				(font
-					(size 1.27 1.27)
-				)
-			)
-		)
-		(property "Datasheet" ""
-			(at 144.78 138.43 0)
-			(hide yes)
-			(show_name no)
-			(do_not_autoplace no)
-			(effects
-				(font
-					(size 1.27 1.27)
-				)
-			)
-		)
-		(property "Description" "Temperature dependent resistor, negative temperature coefficient"
-			(at 144.78 139.7 0)
-			(hide yes)
-			(show_name no)
-			(do_not_autoplace no)
-			(effects
-				(font
-					(size 1.27 1.27)
-				)
-			)
-		)
-		(pin "2"
-		)
-		(pin "1"
-		)
-		(instances
-			(project "Avionics-BatteryBoard"
-				(path "/b6fd875d-6e05-4440-9a05-0f0aa046a0ef/ad142cc2-d77f-4a6c-99c2-d9e17f4c27ae"
-					(reference "TH6")
-					(unit 1)
-				)
-			)
-		)
-	)
-	(symbol
 		(lib_id "power:GND")
 		(at 67.31 109.22 0)
@@
 	(symbol
 		(lib_id "power:GND")
-		(at 144.78 146.05 0)
+		(at 144.78 138.43 0)
 		(unit 1)
 		(body_style 1)
@@
 		(dnp no)
 		(property "Reference" "#PWR052"
-			(at 144.78 152.4 0)
+			(at 144.78 144.78 0)
 			(hide yes)
 			(show_name no)
@@
 		)
 		(property "Value" "SYSTEM_VSS"
-			(at 144.78 149.86 0)
+			(at 144.78 142.24 0)
 			(show_name no)
 			(do_not_autoplace no)
@@
 		)
 		(property "Footprint" ""
-			(at 144.78 146.05 0)
+			(at 144.78 138.43 0)
 			(hide yes)
 			(show_name no)
@@
 		)
 		(property "Datasheet" ""
-			(at 144.78 146.05 0)
+			(at 144.78 138.43 0)
 			(hide yes)
 			(show_name no)
@@
 		)
 		(property "Description" "Power symbol creates a global label with name \"GND\" , ground"
-			(at 144.78 146.05 0)
+			(at 144.78 138.43 0)
 			(hide yes)
 			(show_name no)
@@
 	)
 	(symbol
-		(lib_id "Device:Thermistor_NTC")
-		(at 132.08 139.7 0)
-		(mirror y)
-		(unit 1)
-		(body_style 1)
-		(exclude_from_sim no)
-		(in_bom yes)
-		(on_board yes)
-		(in_pos_files yes)
-		(dnp no)
-		(property "Reference" "TH3"
-			(at 129.54 138.7474 0)
-			(show_name no)
-			(do_not_autoplace no)
-			(effects
-				(font
-					(size 1.27 1.27)
-				)
-				(justify left)
-			)
-		)
-		(property "Value" "10k 3435k"
-			(at 129.54 141.2874 0)
-			(show_name no)
-			(do_not_autoplace no)
-			(effects
-				(font
-					(size 1.27 1.27)
-				)
-				(justify left)
-			)
-		)
-		(property "Footprint" "Capacitor_SMD:C_0603_1608Metric"
-			(at 132.08 138.43 0)
-			(hide yes)
-			(show_name no)
-			(do_not_autoplace no)
-			(effects
-				(font
-					(size 1.27 1.27)
-				)
-			)
-		)
-		(property "Datasheet" ""
-			(at 132.08 138.43 0)
-			(hide yes)
-			(show_name no)
-			(do_not_autoplace no)
-			(effects
-				(font
-					(size 1.27 1.27)
-				)
-			)
-		)
-		(property "Description" "Temperature dependent resistor, negative temperature coefficient"
-			(at 132.08 139.7 0)
-			(hide yes)
-			(show_name no)
-			(do_not_autoplace no)
-			(effects
-				(font
-					(size 1.27 1.27)
-				)
-			)
-		)
-		(pin "2"
-		)
-		(pin "1"
-		)
-		(instances
-			(project "Avionics-BatteryBoard"
-				(path "/b6fd875d-6e05-4440-9a05-0f0aa046a0ef/ad142cc2-d77f-4a6c-99c2-d9e17f4c27ae"
-					(reference "TH3")
-					(unit 1)
-				)
-			)
-		)
-	)
-	(symbol
 		(lib_id "Device:R_Small")
 		(at 46.99 88.9 90)
@@
 	(symbol
 		(lib_id "power:GND")
-		(at 132.08 146.05 0)
+		(at 132.08 138.43 0)
 		(unit 1)
 		(body_style 1)
@@
 		(dnp no)
 		(property "Reference" "#PWR051"
-			(at 132.08 152.4 0)
+			(at 132.08 144.78 0)
 			(hide yes)
 			(show_name no)
@@
 		)
 		(property "Value" "SYSTEM_VSS"
-			(at 132.08 149.86 0)
+			(at 132.08 142.24 0)
 			(show_name no)
 			(do_not_autoplace no)
@@
 		)
 		(property "Footprint" ""
-			(at 132.08 146.05 0)
+			(at 132.08 138.43 0)
 			(hide yes)
 			(show_name no)
@@
 		)
 		(property "Datasheet" ""
-			(at 132.08 146.05 0)
+			(at 132.08 138.43 0)
 			(hide yes)
 			(show_name no)
@@
 		)
 		(property "Description" "Power symbol creates a global label with name \"GND\" , ground"
-			(at 132.08 146.05 0)
+			(at 132.08 138.43 0)
 			(hide yes)
 			(show_name no)
@@
 		)
 		(property "Field5" "NTCS0603E3103JLT"
-			(at 138.43 152.146 0)
-			(show_name no)
-			(do_not_autoplace no)
+			(at 138.43 144.526 0)
+			(show_name no)
+			(do_not_autoplace no)

Commit message: routing
Parts:
- renumbered C7 to C5, C9 to C6, C8 to C7, C10 to C8, C11 to C9, J5 to J2, R49 to R10, R50 to R11, R41 to R12, R44 to R13, R42 to R14, R45 to R15, R46 to R16, R51 to R17, R52 to R18, R53 to R19, R43 to R7, R47 to R8, R48 to R9, TH4 to TH2, TH2 to TH3, TH5 to TH4, U5 to U3
