File: Avionics-BatteryBoard.kicad_sch (KiCad schematic)
At the start: 4 parts

Commit message: More updates
Parts:
- added TP1, TP2: TestPoint, TestPoint:TestPoint_Pad_D1.5mm, symbol Connector:TestPoint
Connections:
- net Battery Bus Protection/CHARGE_ACTIVE: now also TP1.1
- net Battery Bus Protection/DISCHARGE_ACTIVE: now also TP2.1
- no-connect marks 1 -> 0
Other:
- removed sheet IO Expander
- sheet Battery Temperature Protection ports: added HEATER0_ON, HEATER1_ON, HEATER_ENABLE; removed CB-RESET, HEATER_ENABLE0, HEATER_ENABLE1, ON/~{OFF}, ~{FAULT}
- sheet Interfaces ports: added HEAT0_ON, HEAT1_ON, HEATER_ENABLE; removed none
- note removed: "Could put ALERT ON IO5"
- note removed: "Could put all GPIO ON FPC"

Commit message: Finalized updates with recommendations and exported files
Other:
- sheet Interfaces ports: added HEATER0_ON, HEATER1_ON; removed HEAT0_ON, HEAT1_ON
- note added: "EXTERNAL INTERFACES"
Changed lines of the file:
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@@
+		)
+	)
+	(text "EXTERNAL INTERFACES"
+		(exclude_from_sim no)
+		(at 216.662 106.68 90)
+		(effects
+			(font
+				(size 1.905 1.905)
+			)
 		)
 	)
@@
 			)
 		)
-		(pin "HEAT0_ON" output
+		(pin "HEATER1_ON" output
+			(at 185.42 104.14 180)
+			(effects
+				(font
+					(size 1.27 1.27)
+				)
+				(justify left)
+			)
+		)
+		(pin "HEATER0_ON" output
 			(at 185.42 99.06 180)
 			(effects
 				(font
-					(size 1.27 1.27)
-				)
-				(justify left)
-			)
-		)
-		(pin "HEAT1_ON" output
-			(at 185.42 104.14 180)
-			(effects
-				(font

Commit message: v3.1 Updates
Parts:
- H1, H2, H3, H4, TP1, TP2: now left out of the parts list
Changed lines of the file:
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@@
 		(unit 1)
 		(exclude_from_sim no)
-		(in_bom yes)
+		(in_bom no)
 		(on_board yes)
 		(dnp no)
@@
 		(unit 1)
 		(exclude_from_sim no)
-		(in_bom yes)
+		(in_bom no)
 		(on_board yes)
 		(dnp no)
@@
 		(unit 1)
 		(exclude_from_sim no)
-		(in_bom yes)
+		(in_bom no)
 		(on_board yes)
 		(dnp no)
@@
 		(unit 1)
 		(exclude_from_sim no)
-		(in_bom yes)
+		(in_bom no)
 		(on_board yes)
 		(dnp no)
@@
 		(unit 1)
 		(exclude_from_sim no)
-		(in_bom yes)
+		(in_bom no)
 		(on_board yes)
 		(dnp no)
@@
 		(unit 1)
 		(exclude_from_sim no)
-		(in_bom yes)
-		(on_board yes)
-		(dnp no)
+		(in_bom no)
+		(on_board yes)
+		(dnp no)
