File: Avionics-BatteryBoard.kicad_sch (KiCad schematic)
At the start: 6 parts

Commit message: More v3.2 updates
Parts:
- H1, H2, H3, H4: footprint MountingHole:MountingHole_3.2mm_M3_Pad_TopBottom -> MountingHole:MountingHole_3.2mm_M3_Pad_Via
Changed lines of the file:
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@@
 			)
 		)
-		(property "Footprint" "MountingHole:MountingHole_3.2mm_M3_Pad_TopBottom"
+		(property "Footprint" "MountingHole:MountingHole_3.2mm_M3_Pad_Via"
 			(at 250.19 153.67 0)
 			(effects
@@
 			)
 		)
-		(property "Footprint" "MountingHole:MountingHole_3.2mm_M3_Pad_TopBottom"
+		(property "Footprint" "MountingHole:MountingHole_3.2mm_M3_Pad_Via"
 			(at 250.19 147.32 0)
 			(effects
@@
 			)
 		)
-		(property "Footprint" "MountingHole:MountingHole_3.2mm_M3_Pad_TopBottom"
+		(property "Footprint" "MountingHole:MountingHole_3.2mm_M3_Pad_Via"
 			(at 250.19 140.97 0)
 			(effects
@@
 			)
 		)
-		(property "Footprint" "MountingHole:MountingHole_3.2mm_M3_Pad_TopBottom"
+		(property "Footprint" "MountingHole:MountingHole_3.2mm_M3_Pad_Via"
 			(at 250.19 134.62 0)
 			(effects

Commit message: v4.1
Other:
- sheet Battery Temperature Protection ports: added none; removed HEATER_ENABLE
- sheet Interfaces ports: added none; removed HEATER_ENABLE
Changed lines of the file:
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@@
-	(wire
-		(pts
-			(xy 157.48 62.23) (xy 181.61 62.23)
-		)
-		(stroke
-			(width 0)
-			(type default)
-		)
-	)
 	(wire
 		(pts
@@
 	(wire
 		(pts
-			(xy 181.61 93.98) (xy 181.61 62.23)
-		)
-		(stroke
-			(width 0)
-			(type default)
-		)
-	)
-	(wire
-		(pts
 			(xy 119.38 109.22) (xy 66.04 109.22)
 		)
@@
 		(pts
 			(xy 66.04 82.55) (xy 66.04 88.9)
-		)
-		(stroke
-			(width 0)
-			(type default)
-		)
-	)
-	(wire
-		(pts
-			(xy 185.42 93.98) (xy 181.61 93.98)
 		)
 		(stroke
@@
 	)
 	(sheet
-		(at 119.38 59.69)
-		(size 38.1 15.24)
+		(at 119.38 64.77)
+		(size 38.1 10.16)
 		(exclude_from_sim no)
 		(in_bom yes)
@@
 		)
 		(property "Sheetname" "Battery Temperature Protection"
-			(at 119.38 58.9784 0)
+			(at 119.38 64.0584 0)
 			(show_name no)
 			(do_not_autoplace no)
@@
 		(pin "HEATER1_ON" input
 			(at 157.48 72.39 0)
-			(effects
-				(font
-					(size 1.27 1.27)
-				)
-				(justify right)
-			)
-		)
-		(pin "HEATER_ENABLE" input
-			(at 157.48 62.23 0)
 			(effects
 				(font
@@
 	)
 	(sheet
-		(at 185.42 90.932)
-		(size 27.94 30.988)
+		(at 185.42 95.25)
+		(size 27.94 26.67)
 		(exclude_from_sim no)
 		(in_bom yes)
@@
 		)
 		(property "Sheetname" "Interfaces"
-			(at 185.42 90.2204 0)
+			(at 185.42 94.5384 0)
 			(show_name no)
 			(do_not_autoplace no)
@@
 			(effects
 				(font
-					(size 1.27 1.27)
-				)
-				(justify left)
-			)
-		)
-		(pin "HEATER_ENABLE" output
-			(at 185.42 93.98 180)
-			(effects
-				(font
