File: Interfaces.kicad_sch (KiCad schematic)
At the start: 8 parts, among them J6 205338-0002, J7 205338-0004, J8 282834-4, J9 522711069, U6 D5V0P4UR6SO, U7 D5V0P4UR6SO

Commit message: v4.1
Parts:
- added C15: 10u, Capacitor_SMD:C_0805_2012Metric, symbol Device:C_Small
- added J12: QSH-030-01-L-D-A, Argus-Connectors:SAMTEC_QSH-030-01-L-D-A, symbol Argus-Connectors:QSH-030-01-L-D-A
Connections:
- net +3V3: now also C15.1, J12.21, J12.22, J12.23, J12.24
- net ALERT: now also J12.58
- net GND: now also C15.2, J12.11, J12.12, J12.13, J12.14, J12.15, J12.16, J12.17, J12.18, J12.19, J12.20, J12.25, J12.26, J12.27, J12.28, J12.35, J12.41, J12.44, J12.47, J12.59, J12.60, J12.S1 (GND), J12.S2 (GND), J12.S3 (GND), J12.S4 (GND)
- net HEATER0_ON: now also J12.54
- net HEATER1_ON: now also J12.56
- net SCL_BUS: now also J12.37
- net SDA_BUS: now also J12.39
- net HEATER_ENABLE: no longer names the net of U6.6 (IO4)
- net HEATER_ENABLE: no longer J9.1 (Pin_1)
- new net VBATT: J12.01, J12.02, J12.03, J12.04, J12.05, J12.06, J12.07, J12.08, J12.09, J12.10
- no-connect marks 2 -> 25
Other:
- note added: "Samtec to mainboard"
- moved on the sheet: C14, J9, U6, U7
