File: Interfaces.kicad_sch (KiCad schematic)
At the start: 10 parts, among them J12 QSH-030-01-L-D-A, J6 205338-0002, J7 205338-0004, J8 282834-4, J9 522711069, U6 D5V0P4UR6SO, U7 D5V0P4UR6SO

Commit message: making a few changes
Parts:
- removed J12: QSH-030-01-L-D-A, Argus-Connectors:SAMTEC_QSH-030-01-L-D-A, symbol Argus-Connectors:QSH-030-01-L-D-A
- removed U6, U7: D5V0P4UR6SO, Package_TO_SOT_SMD:SOT-23-6, symbol Power_Protection:SRV05-4
- added J10: QTH-030-01-L-D-A, Argus-Connectors:SAMTEC-QTH-030-01-L-D-A, symbol Argus-Connectors:QTH-030-01-L-D-A
Connections:
- net +3V3: now also J10.21, J10.22, J10.23, J10.24
- net ALERT: now also J10.58
- net GND: now also J10.25, J10.26, J10.27, J10.28, J10.35, J10.41, J10.44, J10.47, J10.59, J10.60, J10.G1 (GND), J10.G2 (GND), J10.G3 (GND), J10.G4 (GND)
- net HEATER0_ON: now also J10.54
- net HEATER1_ON: now also J10.56
- net SCL_BUS: now also J10.37
- net SDA_BUS: now also J10.39
- net SYSTEM_VDD: now also J10.1, J10.10, J10.2, J10.3, J10.4, J10.5, J10.6, J10.7, J10.8, J10.9
- net SYSTEM_VSS: now also J10.11, J10.12, J10.13, J10.14, J10.15, J10.16, J10.17, J10.18, J10.19, J10.20
- no-connect marks 25 -> 22
Other:
- title: Argus Batteryboard -> Batteryboard
- moved on the sheet: C15

Commit message: routing
Parts:
- renumbered D6 to D7, J6 to J3, J7 to J4, J8 to J5, J10 to J7, J9 to J8
