File: BatteryTemperatureProtection.kicad_sch (KiCad schematic)
At the start: 9 parts, among them Q1 SIRA99DP-T1-GE3, Q2 IRLML2803, U8 TLX9000

Commit message: v4.1
Parts:
- added U11: 74AUP1G32, Package_TO_SOT_SMD:Texas_R-PDSO-N5_DRL-5, symbol 74xGxx:74AUP1G32
Connections:
- net +3V3: now also U11.5 (VCC)
- net GND: now also U11.3 (GND)
- net HEATER0_ON: now also U11.1
- net HEATER1_ON: now also U11.2
- net HEATER_ENABLE: now also U11.4

Commit message: making a few changes
Parts:
- removed D3: GREEN, LED_SMD:LED_0603_1608Metric, symbol Device:LED_Small
- removed F9: 5A, Fuse:Fuse_1206_3216Metric, symbol Device:Fuse_Small
- removed Q1: SIRA99DP-T1-GE3, Package_SO:PowerPAK_SO-8_Single, symbol Transistor_FET:Si7141DP
- removed Q2: IRLML2803, Package_TO_SOT_SMD:SOT-23, symbol Argus-IC:IRLML2803
- removed R10, R7: 10k, Resistor_SMD:R_0603_1608Metric, symbol Device:R_Small
- removed R8: 1k, Resistor_SMD:R_0603_1608Metric, symbol Device:R_Small
- removed R9: 4k7, Resistor_SMD:R_0603_1608Metric, symbol Device:R_Small
- removed U11: 74AUP1G32, Package_TO_SOT_SMD:Texas_R-PDSO-N5_DRL-5, symbol 74xGxx:74AUP1G32
- removed U8: TLX9000, Package_SO:SOIC-4_4.55x2.6mm_P1.27mm, symbol Isolator:Optocoupler_DC_PhotoNPN_AKEC
Other:
- title: Argus Batteryboard -> Batteryboard
